File: misterydev20k/interfaces.kicad_sch (KiCad schematic)
At the start: 44 parts, among them J4 Micro_SD_Card_Det1, J5 HDMI_A, SW2 KEY1, SW3 KEY2

Commit message: More updates in dev20k
Parts:
- removed R26: 22, Resistor_SMD:R_0402_1005Metric, symbol Device:R_Small
Connections:
- net SD_CLK: now also J4.5 (CLK)
- net VCC33 renamed +3.3V
Other:
- moved on the sheet: R23, R24, R25, R27, R28

Commit message: Update missing files
Parts:
- added R36: 10k, Resistor_SMD:R_0402_1005Metric, symbol Device:R_Small
Connections:
- net +3.3V: now also R36.1
- net ~{SD_DET}: now reaches J4.9 (DET)
- net ~{SD_DET}: now also R36.2
- no-connect marks 2 -> 1
Other:
- moved on the sheet: C45, R23, R24, R25, R27, R28

Commit message: Another board update
Parts:
- removed D6: RB161QS-40, Diode_SMD:D_0402_1005Metric, symbol Device:D_Schottky
- added D18: 1N5819WS, Diode_SMD:D_SOD-323, symbol Diode:1N5819WS
Connections:
- net +3.3V: now also R41.1
- net +5V: now also D18.2 (A)
- net 5V_DVI: now also D18.1 (K)
- net GND: no longer R41.1
Other:
- moved on the sheet: R41
Changed lines of the file:
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@@
 	(wire
 		(pts
-			(xy 227.33 106.68) (xy 233.68 106.68)
+			(xy 231.14 106.68) (xy 233.68 106.68)
 		)
 		(stroke
@@
 	)
 	(symbol
-		(lib_id "Device:D_Schottky")
-		(at 233.68 59.69 180)
-		(unit 1)
-		(exclude_from_sim no)
-		(in_bom yes)
-		(on_board yes)
-		(dnp no)
-		(property "Reference" "D6"
-			(at 230.632 54.864 0)
-			(effects
-				(font
-					(size 1.27 1.27)
-				)
-			)
-		)
-		(property "Value" "RB161QS-40"
-			(at 230.886 56.896 0)
-			(effects
-				(font
-					(size 1.27 1.27)
-				)
-			)
-		)
-		(property "Footprint" "Diode_SMD:D_0402_1005Metric"
-			(at 233.68 59.69 0)
-			(effects
-				(font
-					(size 1.27 1.27)
-				)
-				(hide yes)
-			)
-		)
-		(property "Datasheet" "~"
-			(at 233.68 59.69 0)
-			(effects
-				(font
-					(size 1.27 1.27)
-				)
-				(hide yes)
-			)
-		)
-		(property "Description" "Schottky diode"
-			(at 233.68 59.69 0)
-			(effects
-				(font
-					(size 1.27 1.27)
-				)
-				(hide yes)
-			)
-		)
-		(property "LCSC Part #" "C28646385"
-			(at 233.68 59.69 0)
-			(effects
-				(font
-					(size 1.27 1.27)
-				)
-				(hide yes)
-			)
-		)
-		(pin "1"
-		)
-		(pin "2"
-		)
-		(instances
-			(project "misterydev20k"
-				(path "/ba62e47e-9e07-4e97-ab08-24b670d50f97/1ae93680-6377-49c6-a9eb-78c5d0ac1afd/1f0ce8d2-82e9-428d-82b0-dc1a063a67f6"
-					(reference "D6")
-					(unit 1)
-				)
-			)
-		)
-	)
-	(symbol
 		(lib_name "+3V3_1")
 		(lib_id "power:+3V3")
@@
 	(symbol
 		(lib_id "Device:R_Small")
-		(at 227.33 109.22 180)
+		(at 228.6 106.68 90)
 		(unit 1)
 		(exclude_from_sim no)
@@
 		(dnp no)
 		(property "Reference" "R41"
-			(at 231.14 105.41 0)
+			(at 228.346 104.648 90)
 			(effects
 				(font
@@
 		)
 		(property "Value" "10k"
-			(at 231.14 107.95 0)
+			(at 228.6 108.712 90)
 			(effects
 				(font
@@
 		)
 		(property "Footprint" "Resistor_SMD:R_0402_1005Metric"
-			(at 227.33 109.22 0)
+			(at 228.6 106.68 0)
 			(effects
 				(font
@@
 		)
 		(property "Datasheet" "~"
-			(at 227.33 109.22 0)
+			(at 228.6 106.68 0)
 			(effects
 				(font
@@
 		)
 		(property "Description" ""
-			(at 227.33 109.22 0)
+			(at 228.6 106.68 0)
 			(effects
 				(font
@@
 		)
 		(property "LCSC" ""
-			(at 227.33 109.22 0)
+			(at 228.6 106.68 0)
 			(effects
 				(font
@@
 	)
 	(symbol
-		(lib_id "power:GND")
-		(at 227.33 111.76 0)
-		(unit 1)
-		(exclude_from_sim no)
-		(in_bom yes)
-		(on_board yes)
-		(dnp no)
-		(property "Reference" "#PWR0130"
-			(at 227.33 118.11 0)
-			(effects
-				(font
-					(size 1.27 1.27)
-				)
-				(hide yes)
-			)
-		)
-		(property "Value" "GND"
-			(at 227.33 115.824 0)
-			(effects
-				(font
-					(size 1.27 1.27)
-				)
-			)
-		)
-		(property "Footprint" ""
-			(at 227.33 111.76 0)
-			(effects
-				(font
-					(size 1.27 1.27)
-				)
-				(hide yes)
-			)
-		)
-		(property "Datasheet" ""
-			(at 227.33 111.76 0)
-			(effects
-				(font
-					(size 1.27 1.27)
-				)
-				(hide yes)
-			)
-		)
-		(property "Description" ""
-			(at 227.33 111.76 0)
-			(effects
-				(font
-					(size 1.27 1.27)
-				)
-				(hide yes)
-			)
-		)
-		(pin "1"
-		)
-		(instances
-			(project "misterydev20k"
-				(path "/ba62e47e-9e07-4e97-ab08-24b670d50f97/1ae93680-6377-49c6-a9eb-78c5d0ac1afd/1f0ce8d2-82e9-428d-82b0-dc1a063a67f6"
-					(reference "#PWR0130")
-					(unit 1)
-				)
-			)
-		)
-	)
-	(symbol
 		(lib_id "Device:R_Small")
 		(at 149.86 139.7 180)
@@
 	)
 	(symbol
+		(lib_name "+3V3_1")
+		(lib_id "power:+3V3")
+		(at 226.06 106.68 90)
+		(unit 1)
+		(exclude_from_sim no)
+		(in_bom yes)
+		(on_board yes)
+		(dnp no)
+		(property "Reference" "#PWR017"
+			(at 229.87 106.68 0)
+			(effects
+				(font
+					(size 1.27 1.27)
+				)
+				(hide yes)
+			)
+		)
+		(property "Value" "+3.3V"
+			(at 221.742 109.22 0)
+			(effects
+				(font
+					(size 1.27 1.27)
+				)
+				(justify left)
+			)
+		)
+		(property "Footprint" ""
+			(at 226.06 106.68 0)
+			(effects
+				(font
+					(size 1.27 1.27)
+				)
+				(hide yes)
+			)
+		)
+		(property "Datasheet" ""
+			(at 226.06 106.68 0)
+			(effects
+				(font
+					(size 1.27 1.27)
+				)
+				(hide yes)
+			)
+		)
+		(property "Description" "Power symbol creates a global label with name \"+3V3\""
+			(at 226.06 106.68 0)
+			(effects
+				(font
+					(size 1.27 1.27)
+				)
+				(hide yes)
+			)
+		)
+		(pin "1"
+		)
+		(instances
+			(project "misterydev20k"
+				(path "/ba62e47e-9e07-4e97-ab08-24b670d50f97/1ae93680-6377-49c6-a9eb-78c5d0ac1afd/1f0ce8d2-82e9-428d-82b0-dc1a063a67f6"
+					(reference "#PWR017")
+					(unit 1)
+				)
+			)
+		)
+	)
+	(symbol
 		(lib_id "Connector:Micro_SD_Card_Det1")
 		(at 143.51 82.55 0)
@@
 					(unit 1)
 				)
+			)
+		)
+	)
+	(symbol
+		(lib_id "Diode:1N5819WS")
+		(at 233.68 59.69 0)
+		(mirror y)
+		(unit 1)
+		(exclude_from_sim no)
+		(in_bom yes)
+		(on_board yes)
+		(dnp no)
+		(fields_autoplaced yes)
+		(property "Reference" "D18"
+			(at 233.9975 53.34 0)
+			(effects
+				(font
+					(size 1.27 1.27)
+				)
+			)
+		)
+		(property "Value" "1N5819WS"
+			(at 233.9975 55.88 0)
+			(effects
+				(font
+					(size 1.27 1.27)
+				)
+			)
+		)
+		(property "Footprint" "Diode_SMD:D_SOD-323"
+			(at 233.68 64.135 0)
+			(effects
+				(font
+					(size 1.27 1.27)
+				)
+				(hide yes)
+			)
+		)
+		(property "Datasheet" "https://datasheet.lcsc.com/lcsc/2204281430_Guangdong-Hottech-1N5819WS_C191023.pdf"
+			(at 233.68 59.69 0)
+			(effects
+				(font
+					(size 1.27 1.27)
+				)
+				(hide yes)
+			)
+		)
+		(property "Description" "40V 600mV@1A 1A SOD-323 Schottky Barrier Diodes, SOD-323"
+			(at 233.68 59.69 0)
+			(effects
+				(font
+					(size 1.27 1.27)
+				)
+				(hide yes)
+			)
+		)
+		(pin "1"
+		)
+		(pin "2"
+		)
+		(instances
+			(project ""
+				(path "/ba62e47e-9e07-4e97-ab08-24b670d50f97/1ae93680-6377-49c6-a9eb-78c5d0ac1afd/1f0ce8d2-82e9-428d-82b0-dc1a063a67f6"
+					(reference "D18")
+					(unit 1)
+				)

Commit message: Add grove connector for MIDI/UART
Parts:
- added J6: Grove 1125S-4P, Connector:NS-Tech_Grove_1x04_P2mm_Vertical, symbol Connector:Conn_01x04_Pin
Connections:
- net +5V: now also J6.3 (Pin_3)
- net GND: now also J6.4 (Pin_4)
- new net UART_RX: J6.1 (Pin_1)
- new net UART_TX: J6.2 (Pin_2)

Commit message: Update board
Parts:
- added C40, C58: 100nF, Capacitor_SMD:C_0402_1005Metric, symbol Device:C
- added C59, C60: 100nF, Capacitor_SMD:C_0402_1005Metric, symbol Device:C_Small
- added J11: Joystick 0, Connector_Dsub:DSUB-9_Pins_Horizontal_P2.77x2.84mm_EdgePinOffset7.70mm_Housed_MountingHolesOffset9.12mm, symbol Connector:DE9_Plug_MountingHoles
- added J12: Joystick 1, Connector_Dsub:DSUB-9_Pins_Horizontal_P2.77x2.84mm_EdgePinOffset7.70mm_Housed_MountingHolesOffset9.12mm, symbol Connector:DE9_Plug_MountingHoles
- added RN1, RN2, RN3: R_Pack04, Resistor_SMD:R_Array_Concave_4x0603, symbol Device:R_Pack04
- added U10, U9: 74LCX07, Package_SO:TSSOP-14_4.4x5mm_P0.65mm, symbol 74xx:74LCX07
Connections:
- net +3.3V: now also C59.2, C60.2, U10.14 (VCC), U9.14 (VCC)
- net +5V: now also C40.2, C58.2, J11.7, J12.7, RN1.5 (R4.2), RN1.6 (R3.2), RN1.7 (R2.2), RN1.8 (R1.2), RN2.5 (R4.2), RN2.6 (R3.2), RN2.7 (R2.2), RN2.8 (R1.2), RN3.5 (R4.2), RN3.6 (R3.2), RN3.7 (R2.2), RN3.8 (R1.2)
- net GND: now also C40.1, C58.1, C59.1, C60.1, J11.0 (PAD), J11.8, J12.0 (PAD), J12.8, U10.7 (GND), U9.7 (GND)
- new net: J12.6, RN2.2 (R2.1), U10.11
- new net: J12.9, RN2.1 (R1.1), U10.1
- new net: J11.9, RN2.3 (R3.1), U9.1
- new net: J11.6, RN2.4 (R4.1), U9.11
- new net: J11.3, RN1.2 (R2.1), U9.5
- new net: J12.4, RN3.1 (R1.1), U10.3
- new net: J12.1, RN3.4 (R4.1), U10.13
- new net: J11.4, RN1.1 (R1.1), U9.3
- new net: J11.2, RN1.3 (R3.1), U9.9
- new net: J11.1, RN1.4 (R4.1), U9.13
- new net: J12.3, RN3.2 (R2.1), U10.5
- new net: J12.2, RN3.3 (R3.1), U10.9
- new net JOYA0: U9.12
- new net JOYA1: U9.8
- new net JOYA2: U9.6
- new net JOYA3: U9.4
- new net JOYA4: U9.10
- new net JOYA5: U9.2
- new net JOYB0: U10.12
- new net JOYB1: U10.8
- new net JOYB2: U10.6
- new net JOYB3: U10.4
- new net JOYB4: U10.10
- new net JOYB5: U10.2
- no-connect marks 1 -> 3
Other:
- note added: "BTN1"
- note added: "BTN2"
- note added: "DOWN"
- note added: "LEFT"
- note added: "RIGHT"
- note added: "UP"
- moved on the sheet: C18, C19, C20, C21, C22, C23, C24, C25, C26, C45, D12, D13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

Commit message: Fix dev20k schematic
Other:
- company: (none) -> Till Harbaum
- title: (none) -> MiSTeryDev 20k - Peripherials

Commit message: Update pin table
Other:
- title: MiSTeryDev 20k - Peripherials -> MiSTle - MiSTeryDev20k

Commit message: Further work on the dev20k
Connections:
- net JOYA0: now also U9.2; no longer U9.12
- net JOYA1: now also U9.6; no longer U9.8
- net JOYA2: now also U9.12; no longer U9.6
- net JOYA3: now also U9.10; no longer U9.4
- net JOYA4: now also U9.4; no longer U9.10
- net JOYA5: now also U9.8; no longer U9.2
- net JOYB0: now also U10.8; no longer U10.12
- net JOYB1: now also U10.12; no longer U10.8
- net at J12.6, U10.11: now also RN3.2 (R2.1); no longer RN2.2 (R2.1)
- net at J12.9, U10.1: now also RN1.2 (R2.1); no longer RN2.1 (R1.1)
- net at J12.4, U10.3: now also RN1.1 (R1.1); no longer RN3.1 (R1.1)
- net at RN1.3 (R3.1), U9.9: now also J11.9; no longer J11.2
- net at J12.3, U10.5: now also RN3.4 (R4.1); no longer RN3.2 (R2.1)
- net at J12.2, RN3.3 (R3.1): now also U10.13; no longer U10.9
- new net: J11.3, RN2.1 (R1.1), U9.13
- new net: J11.2, RN2.2 (R2.1), U9.5
- new net: J11.6, RN2.3 (R3.1), U9.3
- new net: J11.1, RN2.4 (R4.1), U9.1
- new net: J11.4, RN1.4 (R4.1), U9.11
- new net: J12.1, RN3.1 (R1.1), U10.9
Other:
- moved on the sheet: RN3, U10D, U10F, U9A, U9B, U9C, U9D, U9E, U9F
