File: misteryshield20k_rpipico_dual_db9/misteryshield20k_rpipico_dual_db9.kicad_pcb (KiCad board)
At the start: 2 copper layers, 100 x 57 mm, 70 parts, among them J1 Joystick, J11 USB_A_Stacked, J12 USB_A_Stacked, J2 Joystick, J3 USB_C_Receptacle_PowerOnly, J4 Conn_01x20_Pin, J5 Conn_01x02_Pin, J7 Conn_01x20_Pin, J8 Conn_01x20_Pin, J9 Conn_01x20_Pin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

Commit message: Add files via upload
Parts:
- moved D1 7.54 mm to (100.6, 51.1)
- moved F1 3.64 mm to (99.0, 55.7)
- moved C10 2.66 mm to (100.6, 66.0)
- moved C11 2.66 mm to (99.8, 62.9)
Connections:
- C10 pad 1: +5V -> Net-(J5-Pin_2)
- C11 pad 1: +5V -> Net-(J5-Pin_2)
- D1 pad 2: +5V -> Net-(D1-A)
- F1 pad 1: Net-(F1-Pad1) -> Net-(D1-A)
- F1 pad 2: +5V -> Net-(J5-Pin_2)
- J3 pad A4: Net-(F1-Pad1) -> Net-(D1-A)
- J3 pad A9: Net-(F1-Pad1) -> Net-(D1-A)
- J3 pad B4: Net-(F1-Pad1) -> Net-(D1-A)
- J3 pad B9: Net-(F1-Pad1) -> Net-(D1-A)
- J5 pad 2: +5V -> Net-(J5-Pin_2)
Routing:
- net Net-(J5-Pin_2): track 0.00 -> 25.8 mm
- net +5V: track 439.5 -> 414.1 mm
- net Net-(D1-A): track 0.00 -> 14.7 mm
- net Net-(F1-Pad1): track 12.0 -> 0.00 mm
- net Net-(J3-CC1): track 10.4 -> 11.8 mm

Commit message: Add files via upload
Parts:
- removed J3: USB_C_Receptacle_PowerOnly, Connector_USB:USB_C_Receptacle_GCT_USB4085
- added U1: USB_C_Receptacle_PowerOnly_6P, TYPE-C-SMD_XUNPU_TYPEC-250C-BRP6, F.Cu at (99.2, 43.2)
- C10: value C_1206 (22µF) -> 22µF; footprint PCM_Capacitor_SMD_AKL:C_1206_3216Metric -> Capacitor_SMD:C_0805_2012Metric
- C11: value C_0603 (100nF) -> 100nF; footprint PCM_Capacitor_SMD_AKL:C_0603_1608Metric -> Capacitor_SMD:C_0805_2012Metric
- D1: value PTVS5V0P1UP -> TVS DIODE 5V
- F1: value Fuse -> Reset Fuse 6V 2A; footprint Fuse:Fuse_1812_4532Metric -> Fuse:Fuse_0805_2012Metric
- R28, R29: value 5.1K -> 5K1; footprint Resistor_SMD:R_0603_1608Metric -> Resistor_SMD:R_0805_2012Metric
- moved R29 13.2 mm to (105.4, 44.1), turned to -90 degrees
- moved R28 12.6 mm to (92.9, 44.1), turned to -90 degrees
- moved C11 4.78 mm to (100.3, 58.1)
- moved C10 4.76 mm to (100.4, 61.2)
- moved F1 3.15 mm to (99.3, 52.5)
- moved D1 2.37 mm to (102.4, 49.6)
- moved C3 1.61 mm to (103.4, 81.7)
- moved J2 0.39 mm to (161.2, 72.7)
Routing:
- net P31: track 136.9 -> 129.9 mm
- net GND: track 27.5 -> 33.2 mm, vias 201 -> 255
- net Net-(U1-CC2): track 11.8 -> 7.05 mm, vias 2 -> 0
- net Net-(J5-Pin_2): track 25.8 -> 30.2 mm
- net Net-(D1-A): track 14.7 -> 11.7 mm
- net +3.3V: track 272.4 -> 271.6 mm
Other:
- board text added: "MiSTeryshield PiPico dual DB9"
- board text added: "MiSTle"
- board text added: "Rev. 1"
- board text removed: "MiSTeryShield20kRPiPicoUSB2DB9"
- board text removed: "Rev. V3"

Commit message: Add files via upload
Parts:
- D1: footprint Diode_SMD:D_SOD-123 -> MiSTeryShield20kRPiPico:SOD-128_L3.7-W2.5-LS4.7-RD
- moved C10 4.31 mm to (102.7, 57.6)
- moved C11 3.62 mm to (102.6, 55.4)
- moved J5 1.50 mm to (99.7, 77.1)
- moved D1 0.71 mm to (102.9, 49.1)
- moved Q10 0.09 mm to (161.3, 42.0)
Routing:
- net +5V: track 414.1 -> 408.9 mm
- net /J2-BTN1: track 21.7 -> 23.1 mm, vias 0 -> 2
- net /J2-RIGHT: track 26.5 -> 27.9 mm, vias 0 -> 2
- net P73: track 127.6 -> 126.9 mm
- net +3.3V: track 271.6 -> 272.1 mm
- net GND: track 33.2 -> 32.9 mm, vias 255 -> 251

Commit message: Add files via upload
Parts:
- added D10: green, LED_SMD:LED_0805_2012Metric, F.Cu at (103.8, 93.4)
- added D5: green, LED_SMD:LED_0805_2012Metric, F.Cu at (92.4, 93.4)
- added D6: green, LED_SMD:LED_0805_2012Metric, F.Cu at (94.8, 93.4)
- added D7: green, LED_SMD:LED_0805_2012Metric, F.Cu at (97.0, 93.4)
- added D8: green, LED_SMD:LED_0805_2012Metric, F.Cu at (99.2, 93.4)
- added D9: green, LED_SMD:LED_0805_2012Metric, F.Cu at (101.6, 93.4)
- added R30: 560, Resistor_SMD:R_0805_2012Metric, F.Cu at (92.7, 86.0)
- added R31: 560, Resistor_SMD:R_0805_2012Metric, F.Cu at (95.0, 86.1)
- added R32: 560, Resistor_SMD:R_0805_2012Metric, F.Cu at (97.2, 86.1)
- added R33: 560, Resistor_SMD:R_0805_2012Metric, F.Cu at (99.4, 86.1)
- added R34: 560, Resistor_SMD:R_0805_2012Metric, F.Cu at (101.5, 86.1)
- added R35: 560, Resistor_SMD:R_0805_2012Metric, F.Cu at (103.8, 86.1)
- moved J5 24.5 mm to (101.2, 52.6)
- moved C10 9.97 mm to (95.0, 51.2), turned to 180 degrees
- moved D2 8.85 mm to (125.3, 93.4)
- moved D3 8.85 mm to (123.1, 93.4)
- moved D4 8.85 mm to (120.8, 93.4)
- moved C11 7.79 mm to (95.1, 53.5), turned to 180 degrees
- moved C1 7.61 mm to (89.6, 93.6), turned to 180 degrees
- moved C3 4.32 mm to (105.5, 77.8), turned to -90 degrees
- moved F1 4.15 mm to (96.9, 49.1), turned to 180 degrees
Connections:
- J4 pad 15: unconnected-(J4-Pin_15-Pad15) -> LED2
- J4 pad 16: unconnected-(J4-Pin_16-Pad16) -> LED5
- J4 pad 17: unconnected-(J4-Pin_17-Pad17) -> LED4
- J4 pad 18: unconnected-(J4-Pin_18-Pad18) -> LED3
- J4 pad 6: unconnected-(J4-Pin_6-Pad6) -> LED0
- J4 pad 7: unconnected-(J4-Pin_7-Pad7) -> LED1
Routing:
- net LED0: track 0.00 -> 31.5 mm, vias 0 -> 1
- net LED1: track 0.00 -> 30.1 mm, vias 0 -> 1
- net Net-(J5-Pin_2): track 29.7 -> 7.81 mm
- net LED5: track 0.00 -> 16.8 mm, vias 0 -> 1
- net LED4: track 0.00 -> 15.2 mm, vias 0 -> 1
- net LED3: track 0.00 -> 14.0 mm, vias 0 -> 1
- net LED2: track 0.00 -> 12.7 mm, vias 0 -> 1
- net P74: track 114.4 -> 107.8 mm
- net P77: track 111.6 -> 105.3 mm
- net Net-(D5-K): track 0.00 -> 5.60 mm
- net Net-(D8-K): track 0.00 -> 5.52 mm
- net Net-(D6-K): track 0.00 -> 5.51 mm
- net Net-(D7-K): track 0.00 -> 5.50 mm
- net Net-(D9-K): track 0.00 -> 5.44 mm
- net Net-(D10-K): track 0.00 -> 5.41 mm
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Other:
- board text added: ">"
- board text added: "Joystick"
- board text added: "Keyboard"
- board text added: "LED0"
- board text added: "LED1"
- board text added: "LED2"
- board text added: "LED3"
- board text added: "LED4"
- board text added: "LED5"
- board text added: "Mouse"
- board text added: "USB"
- board text added: "USB HDMI"

Commit message: Add files via upload
Parts:
- removed D10: green, LED_SMD:LED_0805_2012Metric
- removed R33, R34, R35: 560, Resistor_SMD:R_0805_2012Metric
- added D11: BAT54, PCM_JLCPCB:D_SOT-23, F.Cu at (94.8, 73.0)
- added D19: green, LED_SMD:LED_0805_2012Metric, F.Cu at (117.2, 93.4)
- added D20: green, LED_SMD:LED_0805_2012Metric, F.Cu at (119.4, 93.4)
- D5, D6, D8, D9: value green -> BAT54; footprint LED_SMD:LED_0805_2012Metric -> PCM_JLCPCB:D_SOT-23
- R28, R29: value 5K1 -> 5.1K
- moved R32 26.6 mm to (93.2, 59.8)
- moved D7 24.6 mm to (121.6, 93.4)
- moved R31 20.0 mm to (114.3, 91.4), turned to 180 degrees
- moved D5 16.9 mm to (94.8, 76.7), turned to 180 degrees
- moved D9 14.8 mm to (94.8, 80.2), turned to 180 degrees
- moved D8 10.5 mm to (94.8, 83.8), turned to 180 degrees
- moved C3 10.0 mm to (104.0, 87.8), turned to 90 degrees
- moved R30 7.38 mm to (99.6, 83.4), turned to -90 degrees
- moved D6 5.91 mm to (94.8, 87.5), turned to 180 degrees
- moved C1 5.82 mm to (94.7, 90.8), turned to 0 degrees
- moved D4 3.92 mm to (124.7, 93.4)
- moved D2 3.86 mm to (129.2, 93.4)
- moved D3 3.86 mm to (127.0, 93.4)
- moved C10 0.60 mm to (94.4, 51.2)
- moved C11 0.60 mm to (94.5, 53.5)
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Connections:
- D1 pad 1: GND -> Net-(D1-K)
- D1 pad 2: Net-(D1-A) -> GND
- D5 pad 1: Net-(D5-K) -> Net-(D11-Pad1)
- D5 pad 2: +3.3V -> (no net)
- D6 pad 1: Net-(D6-K) -> Net-(D11-Pad1)
- D6 pad 2: +3.3V -> (no net)
- D8 pad 1: Net-(D8-K) -> Net-(D11-Pad1)
- D8 pad 2: +3.3V -> (no net)
- D9 pad 1: Net-(D9-K) -> Net-(D11-Pad1)
- D9 pad 2: +3.3V -> (no net)
- F1 pad 1: Net-(D1-A) -> Net-(D1-K)
- R30 pad 1: Net-(D5-K) -> Net-(D7-K)
- R30 pad 2: LED0 -> Net-(D11-Pad1)
- R31 pad 1: Net-(D6-K) -> Net-(D19-K)
- R31 pad 2: LED1 -> GND
- R32 pad 1: Net-(D7-K) -> Net-(D20-K)
- R32 pad 2: LED2 -> LED0
- U1 pad A9: Net-(D1-A) -> Net-(D1-K)
- U1 pad B9: Net-(D1-A) -> Net-(D1-K)
Routing:
- net Net-(D20-K): track 0.00 -> 52.1 mm, vias 0 -> 2
- net Net-(D7-K): track 5.50 -> 45.5 mm, vias 0 -> 2
- net Net-(D11-Pad1): track 0.00 -> 25.3 mm
- net LED0: track 31.5 -> 6.65 mm
- net LED1: track 30.1 -> 18.1 mm
- net LED5: track 16.8 -> 4.91 mm
- net Net-(D1-K): track 0.00 -> 11.5 mm
- net Net-(D1-A): track 10.8 -> 0.00 mm
- net LED4: track 15.2 -> 5.10 mm
- net LED3: track 14.0 -> 5.54 mm
- net LED2: track 12.7 -> 5.43 mm
- net Net-(D5-K): track 5.60 -> 0.00 mm
- net Net-(D8-K): track 5.52 -> 0.00 mm
- net Net-(D6-K): track 5.51 -> 0.00 mm
- net Net-(D9-K): track 5.44 -> 0.00 mm
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Other:
- board text added: "Activity"
- board text added: "Core"
- board text added: "DB9"
- board text added: "HDMI"
- board text added: "Power"
- board text added: "USB-C"
- board text removed: ">"
- board text removed: "LED0"
- board text removed: "LED1"
- board text removed: "LED2"
- board text removed: "LED3"
- board text removed: "LED4"
- board text removed: "LED5"
- board text removed: "USB HDMI"

Commit message: Add files via upload
Parts:
- added H5: 2x4 Pinheader horizontal, MiSTeryShield20kRPiPico:HDR-TH_8P-P2.54-H-M-R2-C4-S2.54-N, F.Cu at (123.2, 50.7)
- R30: value 560 -> 470
- moved J5 0.58 mm to (101.8, 52.6)
- moved R18 0.30 mm to (124.1, 76.2)
- moved R19 0.30 mm to (121.8, 76.2)
- moved R20 0.30 mm to (119.5, 76.2)
Connections:
- J4 pad 3: unconnected-(J4-Pin_3-Pad3) -> P75
- J7 pad 3: unconnected-(J7-Pin_3-Pad3) -> /UART_TX
- J8 pad 1: unconnected-(J8-Pin_1-Pad1) -> /Pi_Pico_USB_Hub/PI_UART_TX
- J8 pad 2: unconnected-(J8-Pin_2-Pad2) -> /Pi_Pico_USB_Hub/PI_UART_RX
Routing:
- net GND: track 32.9 -> 79.8 mm, vias 260 -> 235
- net +3.3V: track 270.6 -> 315.9 mm, vias 16 -> 17
- net P75: track 0.00 -> 40.5 mm, vias 0 -> 1
- net +5V: track 408.0 -> 430.8 mm
- net /UART_TX: track 0.00 -> 19.3 mm
- net /Pi_Pico_USB_Hub/PI_UART_RX: track 0.00 -> 17.7 mm
- net /Pi_Pico_USB_Hub/PI_UART_TX: track 0.00 -> 16.6 mm
- net P52: track 100.8 -> 93.9 mm
- net P73: track 126.9 -> 121.8 mm
- net P49: track 119.9 -> 115.8 mm
- net /Pi_Pico_USB_Hub/MISO: track 56.4 -> 52.6 mm
- net /Pi_Pico_USB_Hub/CSN: track 50.4 -> 46.7 mm
- net /Pi_Pico_USB_Hub/UP_D-: track 48.4 -> 44.9 mm
- net /Pi_Pico_USB_Hub/MOSI: track 45.4 -> 41.9 mm
- net Net-(D2-A): track 53.2 -> 50.0 mm
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Other:
- board text added: "+3.3V"
- board text added: "+5V"
- board text added: "DEBUG HEADER"
- board text added: "GND"
- board text added: "PI UART RX"
- board text added: "PI UART TX"
- board text added: "Power Switch Header"
- board text added: "UART RX"
- board text added: "UART TX"
- board text removed: "Power Switch Pinheader"

Commit message: Add files via upload
Routing:
- net GND: vias 235 -> 234
Other:
- board text added: "Development"
- board text added: "FPGA Retro Computing Framework"
