File: misteryshield20k_rpipico_dual_db9/misteryshield20k_rpipico_dual_db9.kicad_pcb (KiCad board)
At the start: 2 copper layers, 100 x 57 mm, 82 parts, among them J1 Joystick, J11 USB_A_Stacked, J12 USB_A_Stacked, J2 Joystick, J4 Conn_01x20_Pin, J5 Conn_01x02_Pin, J7 Conn_01x20_Pin, J8 Conn_01x20_Pin, J9 Conn_01x20_Pin, Q1 2N7002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

Commit message: Add files via upload
Parts:
- added J6: Grove 1125S-4P, Connector:NS-Tech_Grove_1x04_P2mm_Vertical, F.Cu at (105.0, 82.9)
- moved C3 11.0 mm to (94.2, 92.9), turned to 0 degrees
- moved R30 9.09 mm to (99.7, 74.3), turned to 180 degrees
- moved C1 0.45 mm to (94.2, 90.8)
- moved D11 0.42 mm to (94.3, 73.0)
- moved D5 0.42 mm to (94.3, 76.7)
- moved D6 0.42 mm to (94.3, 87.5)
- moved D8 0.42 mm to (94.3, 83.8)
- moved D9 0.42 mm to (94.3, 80.2)
Connections:
- J7 pad 17: unconnected-(J7-Pin_17-Pad17) -> MIDI_RX
- J7 pad 18: unconnected-(J7-Pin_18-Pad18) -> MIDI_TX
Routing:
- net Net-(D7-K): track 45.5 -> 33.4 mm
- net +3.3V: track 315.9 -> 327.6 mm
- net +5V: track 430.8 -> 439.1 mm, vias 10 -> 11
- net MIDI_TX: track 0.00 -> 8.22 mm
- net MIDI_RX: track 0.00 -> 4.39 mm
- net P74: track 108.4 -> 104.7 mm
- net GND: track 79.8 -> 83.1 mm, vias 234 -> 243
- net P77: track 105.3 -> 102.7 mm
- net Net-(D11-Pad1): track 25.3 -> 23.1 mm
- net LED2: track 5.43 -> 4.81 mm
Other:
- board text added: "MIDI"
- board text removed: "HDMI"

Commit message: Add files via upload
Parts:
- moved R30 4.22 mm to (100.1, 78.5)
- moved J5 0.62 mm to (102.4, 52.6)
Routing:
- net Net-(D7-K): track 33.4 -> 36.3 mm
- net Net-(J5-Pin_2): track 8.94 -> 9.57 mm
- net +5V: track 439.1 -> 438.5 mm
- net GND: vias 243 -> 246
Other:
- board text added: "Circuit Design by Vossstef PCB Design by Cantclosevi Modifications by Manger"

Commit message: Add files via upload
Parts:
- moved C10 0.60 mm to (95.0, 51.2)
- moved C11 0.60 mm to (95.1, 53.5)
- moved F1 0.60 mm to (96.9, 49.1)
- moved Q8 0.13 mm to (161.3, 49.0)
Routing:
- net GND: track 83.1 -> 14.2 mm, vias 246 -> 243
- net Net-(D7-K): track 36.3 -> 35.1 mm
- net P52: track 93.9 -> 95.0 mm
- net Net-(J5-Pin_2): track 9.57 -> 8.50 mm
- net /Pi_Pico_USB_Hub/PI_UART_TX: track 16.6 -> 17.3 mm
- net Net-(D20-K): track 52.2 -> 51.5 mm
- net +5V: track 438.5 -> 439.1 mm
- net Net-(D1-K): track 11.1 -> 10.5 mm
- net P74: track 104.7 -> 104.1 mm

Commit message: Add files via upload
Parts:
- moved D1 0.94 mm to (102.4, 48.3)
- moved F1 0.94 mm to (96.4, 48.3)
- moved R32 0.87 mm to (93.2, 60.7)
- moved J5 0.85 mm to (102.1, 51.8)
- moved C10 0.53 mm to (95.4, 50.9)
- moved C11 0.49 mm to (95.4, 53.1)
- moved D11 0.30 mm to (94.0, 73.0)
- moved D5 0.30 mm to (94.0, 76.7)
- moved D6 0.30 mm to (94.0, 87.5)
- moved D8 0.30 mm to (94.0, 83.8)
- moved D9 0.30 mm to (94.0, 80.2)
- moved J6 0.20 mm to (104.8, 82.9)
- moved R31 0.20 mm to (114.3, 91.6)
Routing:
- net +5V: track 439.1 -> 401.8 mm, vias 11 -> 10
- net P73: track 122.1 -> 101.2 mm
- net /UART_TX: track 19.1 -> 23.2 mm
- net +3.3V: track 327.5 -> 324.9 mm
- net Net-(D11-Pad1): track 23.5 -> 25.1 mm
- net P31: track 129.7 -> 128.4 mm
- net GND: track 14.2 -> 15.3 mm, vias 243 -> 248
- net /Pi_Pico_USB_Hub/RECONFGN: track 30.3 -> 31.4 mm
- net P77: track 102.6 -> 101.5 mm
- net P52: track 95.0 -> 94.1 mm
- net P75: track 40.5 -> 39.7 mm
- net Net-(D1-K): track 10.5 -> 9.72 mm
- net Net-(D20-K): track 51.5 -> 50.8 mm
- net P49: track 115.8 -> 115.2 mm
Other:
- board text added: "Modifications by Manger"
- board text added: "Original Circuit Design by Vossstef"
- board text added: "Original PCB Design by Cantclosevi"
- board text added: "PI RX"
- board text added: "PI TX"
- board text added: "TN RX"
- board text added: "TN TX"
- board text added: "UART"
- board text removed: "Circuit Design by Vossstef PCB Design by Cantclosevi Modifications by Manger"
- board text removed: "PI UART RX"
- board text removed: "PI UART TX"
- board text removed: "UART RX"
- board text removed: "UART TX"

Commit message: Add files via upload
Parts:
- moved R31 7.33 mm to (117.3, 84.9), turned to 90 degrees
- moved R28 1.02 mm to (93.0, 43.1), turned to 90 degrees
- moved R29 0.99 mm to (105.4, 43.1), turned to 90 degrees
- moved R18 0.90 mm to (123.8, 75.4)
- moved R19 0.90 mm to (121.5, 75.4)
- moved R20 0.90 mm to (119.2, 75.4)
- moved C11 0.48 mm to (95.9, 53.1)
Routing:
- net Net-(D19-K): track 2.30 -> 6.96 mm
- net P73: track 101.2 -> 102.1 mm
- net +3.3V: track 324.9 -> 325.8 mm
- net P31: track 128.4 -> 129.2 mm
- net Net-(D3-K): track 18.5 -> 19.2 mm
- net Net-(D4-K): track 18.3 -> 19.0 mm
- net Net-(D2-K): track 18.9 -> 19.6 mm
- net GND: vias 248 -> 250
Other:
- board text added: "POWER"
- board text added: "RX"
- board text added: "TX"

Commit message: Add files via upload
Parts:
- moved R30 1.67 mm to (98.7, 77.6)
- moved R32 1.11 mm to (93.5, 59.6), turned to 135 degrees
Routing:
- net +5V: track 401.9 -> 397.3 mm
- net +3.3V: track 325.8 -> 323.2 mm
- net Net-(D11-Pad1): track 25.1 -> 23.7 mm
- net LED0: track 6.35 -> 5.46 mm
- net /J2-RIGHT: track 27.9 -> 28.4 mm
Other:
- board text added: "GOWIN"
- board text added: "RASPBERRY"
