File: misteryshield20k_rpipico_dual_db9/misteryshield20k_rpipico_dual_db9.kicad_pcb (KiCad board)
At the start: 2 copper layers, 100 x 57 mm, 83 parts, among them J1 Joystick, J11 USB_A_Stacked, J12 USB_A_Stacked, J2 Joystick, J4 Conn_01x20_Pin, J5 Conn_01x02_Pin, J6 Grove 1125S-4P, J7 Conn_01x20_Pin, J8 Conn_01x20_Pin, J9 Conn_01x20_Pin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

Commit message: Add files via upload
Routing:
- net +5V: track 397.3 -> 395.6 mm
- net +3.3V: track 323.2 -> 322.3 mm
- net GND: vias 250 -> 249
Other:
- board text added: "Design based on the MiSTeryshield"
- board text added: "M5 UART"
- board text added: "PiPico USB, added features"
- board text added: "and modifications by Manger"
- board text removed: "Modifications by Manger"
- board text removed: "Original Circuit Design by Vossstef"
- board text removed: "Original PCB Design by Cantclosevi"

Commit message: Add files via upload
Parts:
- H5: value 2x4 Pinheader horizontal -> 2x3 Pinheader horizontal; footprint MiSTeryShield20kRPiPico:HDR-TH_8P-P2.54-H-M-R2-C4-S2.54-N -> Connector_PinHeader_2.54mm:PinHeader_2x03_P2.54mm_Horizontal
- moved H5 2.67 mm to (120.9, 52.0), turned to 90 degrees
- moved R29 0.17 mm to (105.4, 42.9)
- moved R28 0.15 mm to (93.0, 42.9)
Connections:
- H5 pad 1: /Pi_Pico_USB_Hub/PI_UART_TX -> GND
- H5 pad 2: /Pi_Pico_USB_Hub/PI_UART_RX -> GND
- H5 pad 5: unconnected-(H5-Pad5) -> /Pi_Pico_USB_Hub/PI_UART_RX
- H5 pad 6: GND -> /Pi_Pico_USB_Hub/PI_UART_TX
Routing:
- net +3.3V: track 322.3 -> 276.8 mm, vias 17 -> 16
- net +5V: track 395.6 -> 369.9 mm
- net /UART_TX: track 23.2 -> 17.0 mm
- net GND: track 15.3 -> 20.9 mm, vias 249 -> 349
- net Net-(D1-K): track 9.72 -> 12.0 mm
- net P49: track 115.4 -> 113.7 mm
- net Net-(D7-K): track 35.3 -> 36.9 mm
- net P75: track 39.7 -> 38.4 mm
- net /Pi_Pico_USB_Hub/PI_UART_RX: track 18.1 -> 17.3 mm
Other:
- board text removed: "+3.3V"

Commit message: Add files via upload
Parts:
- removed D11, D6, D8, D9: BAT54, PCM_JLCPCB:D_SOT-23
- removed D19: green, LED_SMD:LED_0805_2012Metric
- D2, D3, D4: value green -> orange
- D5: value BAT54 -> red; footprint PCM_JLCPCB:D_SOT-23 -> LED_SMD:LED_0805_2012Metric
- D7: value green -> yellow
- R31: value 560 -> 470
- moved D5 28.6 mm to (117.2, 93.4), turned to -90 degrees
- moved R31 24.5 mm to (93.3, 79.9), turned to 135 degrees
- moved R30 15.6 mm to (94.8, 62.5), turned to 135 degrees
- moved R32 0.66 mm to (93.2, 59.1)
Connections:
- D5 pad 1: Net-(D11-Pad1) -> Net-(D5-K)
- D5 pad 2: (no net) -> +3.3V
- R30 pad 2: Net-(D11-Pad1) -> LED1
- R31 pad 1: Net-(D19-K) -> Net-(D5-K)
- R31 pad 2: GND -> LED2
Routing:
- net Net-(D5-K): track 0.00 -> 29.7 mm
- net Net-(D11-Pad1): track 23.7 -> 0.00 mm
- net LED1: track 17.4 -> 6.85 mm, vias 1 -> 0
- net Net-(D7-K): track 36.9 -> 47.2 mm
- net Net-(D20-K): track 50.4 -> 59.5 mm, vias 2 -> 0
- net Net-(D19-K): track 6.96 -> 0.00 mm
- net LED3: track 5.37 -> 0.00 mm, vias 1 -> 0
- net LED4: track 4.68 -> 0.00 mm, vias 1 -> 0
- net LED5: track 4.54 -> 0.00 mm, vias 1 -> 0
- net GND: track 20.9 -> 18.4 mm, vias 349 -> 347
- net P77: track 101.2 -> 99.6 mm, vias 3 -> 2
- net /IO_DOWN: track 28.7 -> 27.2 mm, vias 0 -> 1
- net P31: track 129.2 -> 128.5 mm
- net P73: track 102.1 -> 101.6 mm, vias 3 -> 2
- net P52: track 94.1 -> 93.7 mm, vias 2 -> 1
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Other:
- board text added: "F.Disk"
- board text added: "H.Disk"
- board text removed: "Activity"
- board text removed: "Core"

Commit message: Add files via upload
Parts:
- D2, D3, D4, D5: footprint LED_SMD:LED_0805_2012Metric -> MiSTeryShield20kRPiPico:LED0805-RD
- D6: renamed from D7; value yellow -> green; footprint LED_SMD:LED_0805_2012Metric -> MiSTeryShield20kRPiPico:LED0805-RD
- D7: renamed from D20; value green -> yellow; footprint LED_SMD:LED_0805_2012Metric -> MiSTeryShield20kRPiPico:LED0805-RD
- J1, J2: footprint Connector_Dsub:DSUB-9_Male_Horizontal_P2.77x2.84mm_EdgePinOffset7.70mm_Housed_MountingHolesOffset9.12mm -> MiSTeryShield20kRPiPico:DSUB-TH_DMR-9P
- moved J1 5.72 mm to (81.2, 67.1), turned to 180 degrees
- moved J2 5.66 mm to (162.6, 67.2), turned to 0 degrees
Connections:
- D6 pad 1: Net-(D7-K) -> Net-(D6-K)
- D7 pad 1: Net-(D20-K) -> Net-(D7-K)
- R32 pad 1: Net-(D20-K) -> Net-(D6-K)
- U1 pad 1: unconnected-(U1-Pad1) -> GND
- U1 pad 2: unconnected-(U1-Pad2) -> GND
- U1 pad 3: unconnected-(U1-Pad3) -> GND
- U1 pad 4: unconnected-(U1-Pad4) -> GND
Routing:
- net Net-(D20-K): track 59.5 -> 0.00 mm
- net Net-(D6-K): track 0.00 -> 58.6 mm
- net GND: track 18.4 -> 7.09 mm, vias 347 -> 330
- net P49: track 113.7 -> 121.6 mm
- net Net-(D7-K): track 47.2 -> 52.2 mm, vias 2 -> 0
- net +3.3V: track 276.8 -> 271.8 mm
- net P77: track 99.6 -> 104.0 mm
- net P31: track 128.5 -> 125.3 mm
- net P52: track 93.7 -> 91.5 mm
- net Net-(D5-K): track 29.7 -> 31.7 mm
- net P73: track 101.6 -> 103.0 mm
- net Net-(U1-CC2): track 7.54 -> 8.39 mm
- net Net-(U1-CC1): track 7.51 -> 8.34 mm
- net /UP: track 16.4 -> 17.2 mm
- net /Pi_Pico_USB_Hub/UP_D+: track 46.4 -> 47.1 mm
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
Commit message: Add files via upload
Parts:
- J6: value Grove 1125S-4P -> S4B-PH-K-S_LF__SN (Grove 1125S-4P); footprint Connector:NS-Tech_Grove_1x04_P2mm_Vertical -> MiSTeryShield20kRPiPico:SHDRRA4W50P0X200_1X4_990X760X480P
- R18, R19, R20: value 560 -> 510
- R31: value 470 -> 560
- R32: value 560 -> 430
- moved J6 6.83 mm to (98.0, 82.9), turned to 180 degrees
- moved C1 4.35 mm to (93.8, 86.5), turned to -45 degrees
- moved C3 3.40 mm to (93.3, 89.6), turned to -45 degrees
- moved R32 0.45 mm to (92.9, 58.8)
- moved R30 0.45 mm to (94.4, 62.3)
Connections:
- J6 pad 1: MIDI_RX -> GND
- J6 pad 2: MIDI_TX -> +5V
- J6 pad 3: +5V -> MIDI_TX
- J6 pad 4: GND -> MIDI_RX
Routing:
- net +5V: track 369.8 -> 374.9 mm
- net +3.3V: track 271.8 -> 274.3 mm
- net P31: track 125.3 -> 126.9 mm
- net Net-(D7-K): track 52.2 -> 53.6 mm
- net Net-(D6-K): track 58.6 -> 59.8 mm
- net /J2-RIGHT: track 28.6 -> 27.5 mm
- net LED0: track 5.23 -> 4.29 mm
- net MIDI_TX: track 8.15 -> 9.04 mm
- net MIDI_RX: track 4.59 -> 5.43 mm
- net LED1: track 6.85 -> 6.13 mm
- net P74: track 103.9 -> 103.4 mm
- net GND: vias 330 -> 323
Other:
- board text added: "DEBUG"
- board text added: "Design based on MiSTeryshield"
- board text added: "HEADER"
- board text added: "PiPico USB : added features"
- board text removed: "DEBUG HEADER"
- board text removed: "Design based on the MiSTeryshield"
- board text removed: "PiPico USB, added features"
