File: misteryshield20k_rpipico_dual_db9/misteryshield20k_rpipico_dual_db9.kicad_sch (KiCad schematic)
At the start: 67 parts, among them J1 Joystick, J2 Joystick, J4 Conn_01x20_Pin, J5 Conn_01x02_Pin, J6 Grove 1125S-4P, J7 Conn_01x20_Pin, Q1 2N7002, Q10 2N7002, Q11 2N7002, Q12 2N7002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

Commit message: Add files via upload
Changed lines of the file:
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@@
 	(wire
 		(pts
-			(xy 233.68 33.02) (xy 240.03 33.02)
+			(xy 228.6 33.02) (xy 240.03 33.02)
 		)
 		(stroke
@@
 	(label "J2-BTN2"
 		(at 38.735 109.22 0)
+		(effects
+			(font
+				(size 1.27 1.27)
+			)
+			(justify left bottom)
+		)
+	)
+	(label "UART_RX"
+		(at 229.87 33.02 0)
 		(effects
 			(font
@@
 	(global_label "P75"
 		(shape bidirectional)
-		(at 233.68 33.02 180)
+		(at 228.6 33.02 180)
 		(fields_autoplaced yes)
 		(effects
@@
 		)
 		(property "Intersheetrefs" "${INTERSHEET_REFS}"
-			(at 225.8945 33.02 0)
-			(effects
-				(font
+			(at 220.8145 33.02 0)
+			(effects
+				(font

Commit message: Add files via upload
Parts:
- J6: Info (none) -> Seeed Technology GROVE 2MM 4PIN R/A CONN horizontal; now not fitted
Other:
- note added: "2nd DB9 Port Mod"
- note added: "Board Power Circuit Mod"
- note added: "FPGA LED Array Mod"
- note added: "MIDI Connector Mod"
- note added: "Tang Nano 20K"
- note removed: "Board Power Circuit"
- note removed: "FPGA LED Array"
- note removed: "MIDI Connector"
- moved on the sheet: D11, D19, D20, D5, D6, D7, D8, D9, J2, Q10, Q11, Q12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

Commit message: Add files via upload
Parts:
- removed D11, D5, D6, D8, D9: BAT54, PCM_JLCPCB:D_SOT-23, symbol PCM_JLCPCB-Diodes:Schottky,BAT54
- removed D19: green, LED_SMD:LED_0805_2012Metric, symbol Device:LED
- added D5: red, LED_SMD:LED_0805_2012Metric, symbol Device:LED
- D7: value green -> yellow; LCSC Part # C2297 -> C2296
- R31: value 560 -> 470
Connections:
- net +3.3V: now also D5.2 (A)
- net GND: no longer R31.2
- net LED1: now also R30.2
- net LED2: now also R31.2
- net at R31.1: now also D5.1 (K)
Other:
- note added: "FDD"
- note added: "HDD"
- note added: "Power"
- note removed: "Board Power"
- note removed: "Core Power"
- note removed: "Drive Activity"
- moved on the sheet: D20, D7, R30, R32

Commit message: Add files via upload
Parts:
- removed J1, J2: Joystick, Connector_Dsub:DSUB-9_Male_Horizontal_P2.77x2.84mm_EdgePinOffset7.70mm_Housed_MountingHolesOffset9.12mm, symbol Connector:DE9_Plug_MountingHoles
- added J1, J2: Joystick, MiSTeryShield20kRPiPico:DSUB-TH_DMR-9P, symbol MiSTeryShield20kRPiPico:DMR-9P
- D5, D7: footprint LED_SMD:LED_0805_2012Metric -> MiSTeryShield20kRPiPico:LED0805-RD; JLC_3DModel_Q (none) -> 23093642268545519703b953fc993978; JLC_3D_Size (none) -> 2.02 1.25
- D6: renamed from D20; footprint LED_SMD:LED_0805_2012Metric -> MiSTeryShield20kRPiPico:LED0805-RD; JLC_3DModel_Q (none) -> 23093642268545519703b953fc993978; JLC_3D_Size (none) -> 2.02 1.25
Connections:
- net +5V: now also J1.7, J2.7
- net BTN1: now also J1.6
- net BTN2: now also J1.9
- net DOWN: now also J1.2
- net GND: now also U1.1, U1.2, U1.3, U1.4, J1.10 (MH1), J1.11 (MH2), J1.8, J2.10 (MH1), J2.11 (MH2), J2.8
- net J2-BTN1: now also J2.6
- net J2-BTN2: now also J2.9
- net J2-DOWN: now also J2.2
- net J2-LEFT: now also J2.3
- net J2-RIGHT: now also J2.4
- net J2-UP: now also J2.1
- net LEFT: now also J1.3
- net RIGHT: now also J1.4
- net UP: now also J1.1
- no-connect marks 12 -> 8
Other:
- moved on the sheet: Q10, Q11, Q12, Q7, Q8, Q9, R11, R14, R15, R16, R17, R21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

Commit message: Add files via upload
Parts:
- removed J6: Grove 1125S-4P, Connector:NS-Tech_Grove_1x04_P2mm_Vertical, symbol Connector:Conn_01x04_Pin
- added J6: S4B-PH-K-S_LF__SN (Grove 1125S-4P), MiSTeryShield20kRPiPico:SHDRRA4W50P0X200_1X4_990X760X480P, symbol MiSTeryShield20kRPiPico:S4B-PH-K-S_LF__SN_
- D1: JLCPCB Part # C426873 -> C83329
- D5: LCSC (none) -> C2295
- D7: LCSC (none) -> C2296
- R30: LCSC Part # C28636 -> C17710
- R31: value 470 -> 560
- R32: value 560 -> 430; LCSC Part # C28636 -> C42000
Connections:
- net +5V: now also J6.2
- net GND: now also J6.1
- net MIDI_RX: now also J6.4
- net MIDI_TX: now also J6.3
Other:
- moved on the sheet: C10, C11, D1, F1, J5, R28, R29, U1

Commit message: Add files via upload
Parts:
- D1: footprint MiSTeryShield20kRPiPico:SOD-128_L3.7-W2.5-LS4.7-RD -> MiSTeryShield20kRPiPico:SOD-123_L2.7-W1.6-LS3.7-RD; Bemerkung PTVS5V0P1UP -> (none); JLCPCB Part # C83329 -> (none); LCSC Part # (none) -> C83329
- J1, J2: value Joystick -> D-DMR009PM-D002; LCSC Part #  (none) -> C141880; LCSC Part Name DMR9公 -> (none); Manufacturer Ckmtw(灿科盟) -> (none); Manufacturer Part D-DMR009PM-D002 -> (none); Supplier LCSC -> (none); Supplier Part C141880 -> (none)
- J4, J7: footprint Connector_PinSocket_2.54mm:PinSocket_1x20_P2.54mm_Vertical -> MiSTeryShield20kRPiPico:PinSocket_1x20_P2.54mm_Vertical; Comment 1x20, P2.54mm -> (none)
- J5: footprint Connector_PinHeader_2.54mm:PinHeader_1x02_P2.54mm_Horizontal -> MiSTeryShield20kRPiPico:HDR-TH_2P-P2.54-H-M-W10.4
- J6: value S4B-PH-K-S_LF__SN (Grove 1125S-4P) -> Grove 1125S-4P
Connections:
- net +5V: now also J5.2 (Pin_2); no longer J5.1 (Pin_1)
- net at C10.1, C11.1, F1.2: now also J5.1 (Pin_1); no longer J5.2 (Pin_2)
Other:
- note added: "2nd DB9 Port (Mod)"
- note added: "Board Power Circuit (Mod)"
- note added: "FPGA LED Array (Mod)"
- note added: "MIDI Connector (Mod)"
- note removed: "2nd DB9 Port Mod"
- note removed: "Board Power Circuit Mod"
- note removed: "FPGA LED Array Mod"
- note removed: "MIDI Connector Mod"
- moved on the sheet: J5
Changed lines of the file:
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@@
 		)
 	)
-	(text "Board Power Circuit Mod"
+	(text "Board Power Circuit (Mod)"
 		(exclude_from_sim no)
-		(at 171.45 121.92 0)
+		(at 175.26 124.46 0)
 		(effects
 			(font
@@
 		)
 	)
-	(text "MIDI Connector Mod"
+	(text "MIDI Connector (Mod)"
 		(exclude_from_sim no)
-		(at 232.41 87.63 0)
+		(at 237.49 87.63 0)
 		(effects
 			(font
@@
 		)
 	)
-	(text "2nd DB9 Port Mod"
+	(text "2nd DB9 Port (Mod)"
 		(exclude_from_sim no)
-		(at 30.48 91.44 0)
+		(at 29.21 91.44 0)
 		(effects
 			(font
@@
 		)
 	)
-	(text "FPGA LED Array Mod"
+	(text "FPGA LED Array (Mod)"
 		(exclude_from_sim no)
-		(at 112.522 148.59 0)
+		(at 113.03 148.59 0)
 		(effects
 			(font
@@
 			)
 		)
-		(property "Value" "Joystick"
+		(property "Value" "D-DMR009PM-D002"
 			(at 30.48 44.45 0)
 			(effects
@@
 			)
 		)
-		(property "Datasheet" "https://item.szlcsc.com/datasheet/D-DMR009PM-D002/153211.html"
-			(at 30.48 59.69 0)
-			(effects
-				(font
-					(size 1.27 1.27)
-				)
-				(hide yes)
-			)
-		)
-		(property "Description" "Connector Type:Standard D-Sub Gender:Male Number of Pins:9P Mounting Type:Right Angle Number of Rows:2 Current Rating-Signal:3A Current Rating-Power:- Voltage Rating:- Color:Black Operating Temperature:-50°C~+105°C Operating Temperature:-50°C~+105°C"
-			(at 30.48 59.69 0)
-			(effects
-				(font
-					(size 1.27 1.27)
-				)
-				(hide yes)
-			)
-		)
-		(property "Manufacturer Part" "D-DMR009PM-D002"
-			(at 30.48 59.69 0)
-			(effects
-				(font
-					(size 1.27 1.27)
-				)
-				(hide yes)
-			)
-		)
-		(property "Manufacturer" "Ckmtw(灿科盟)"
-			(at 30.48 59.69 0)
-			(effects
-				(font
-					(size 1.27 1.27)
-				)
-				(hide yes)
-			)
-		)
-		(property "Supplier Part" "C141880"
+		(property "Datasheet" ""
 			(at 30.48 59.69 0)
 			(effects
@@
 			)
 		)
-		(property "Supplier" "LCSC"
+		(property "Description" ""
 			(at 30.48 59.69 0)
 			(effects
@@
 			)
 		)
-		(property "LCSC Part Name" "DMR9公"
+		(property "LCSC Part # " "C141880"
 			(at 30.48 59.69 0)
 			(effects
@@
 			)
 		)
-		(property "Footprint" "MiSTeryShield20kRPiPico:SOD-128_L3.7-W2.5-LS4.7-RD"
+		(property "Footprint" "MiSTeryShield20kRPiPico:SOD-123_L2.7-W1.6-LS3.7-RD"
 			(at 222.25 138.43 0)
 			(effects
@@
 			)
 		)
-		(property "Datasheet" "https://www.tme.eu/Document/475226a1f5f23e88222b181b564f5c39/PTVSXP1UP_SER.pdf"
+		(property "Datasheet" ""
 			(at 222.25 138.43 0)
 			(effects
@@
 			)
 		)
-		(property "Description" "SOD-128 Unidirectional TVS diode, 5V, 600W, Alternate KiCAD Library"
+		(property "Description" ""
 			(at 222.25 138.43 0)
 			(effects
@@
 			)
 		)
-		(property "JLCPCB Part #" "C83329"
-			(at 222.25 138.43 90)
-			(effects
-				(font
-					(size 1.27 1.27)
-				)
-				(hide yes)
-			)
-		)
-		(property "Bemerkung" "PTVS5V0P1UP"
-			(at 222.25 138.43 90)
+		(property "LCSC Part #" "C83329"
+			(at 222.25 138.43 0)
 			(effects
 				(font
@@
 			)
 		)
-		(property "Value" "S4B-PH-K-S_LF__SN (Grove 1125S-4P)"
+		(property "Value" "Grove 1125S-4P"
 			(at 253.746 108.458 0)
 			(effects
@@
 			)
 		)
-		(property "Footprint" "Connector_PinSocket_2.54mm:PinSocket_1x20_P2.54mm_Vertical"
-			(at 191.77 54.61 0)
-			(effects
-				(font
-					(size 1.27 1.27)
-				)
-				(hide yes)
-			)
-		)
-		(property "Datasheet" "~"
+		(property "Footprint" "MiSTeryShield20kRPiPico:PinSocket_1x20_P2.54mm_Vertical"
 			(at 191.77 54.61 0)
 			(effects
@@
 			)
 		)
-		(property "Description" "Generic connector, single row, 01x20, script generated"
-			(at 191.77 54.61 0)
-			(effects
-				(font
-					(size 1.27 1.27)
-				)
-				(hide yes)
-			)
-		)
-		(property "JLCPCB Position Offset" ""
+		(property "Datasheet" ""
 			(at 191.77 54.61 0)
 			(effects
@@
 			)
 		)
-		(property "JLCPCB Rotation Offset" ""
+		(property "Description" ""
 			(at 191.77 54.61 0)
 			(effects
@@
 			)
 		)
-		(property "Comment" "1x20, P2.54mm"
-			(at 191.77 54.61 0)
-			(effects
-				(font
-					(size 1.27 1.27)
-				)
-				(hide yes)
-			)
-		)
 		(pin "1"
 		)
@@
 			)
 		)
-		(property "Value" "Joystick"
+		(property "Value" "D-DMR009PM-D002"
 			(at 33.02 105.41 0)
 			(effects
@@
 			)
 		)
-		(property "Datasheet" "https://item.szlcsc.com/datasheet/D-DMR009PM-D002/153211.html"
-			(at 33.02 120.65 0)
-			(effects
-				(font
-					(size 1.27 1.27)
-				)
-				(hide yes)
-			)
-		)
-		(property "Description" "Connector Type:Standard D-Sub Gender:Male Number of Pins:9P Mounting Type:Right Angle Number of Rows:2 Current Rating-Signal:3A Current Rating-Power:- Voltage Rating:- Color:Black Operating Temperature:-50°C~+105°C Operating Temperature:-50°C~+105°C"
-			(at 33.02 120.65 0)
-			(effects
-				(font
-					(size 1.27 1.27)
-				)
-				(hide yes)
-			)
-		)
-		(property "Manufacturer Part" "D-DMR009PM-D002"
-			(at 33.02 120.65 0)
-			(effects
-				(font
-					(size 1.27 1.27)
-				)
-				(hide yes)
-			)
-		)
-		(property "Manufacturer" "Ckmtw(灿科盟)"
-			(at 33.02 120.65 0)
-			(effects
-				(font
-					(size 1.27 1.27)
-				)
-				(hide yes)
-			)
-		)
-		(property "Supplier Part" "C141880"
+		(property "Datasheet" ""
 			(at 33.02 120.65 0)
 			(effects
@@
 			)
 		)
-		(property "Supplier" "LCSC"
+		(property "Description" ""
 			(at 33.02 120.65 0)
 			(effects
@@
 			)
 		)
-		(property "LCSC Part Name" "DMR9公"
+		(property "LCSC Part # " "C141880"
 			(at 33.02 120.65 0)
 			(effects
@@
 			)
 		)
-		(property "Footprint" "Connector_PinSocket_2.54mm:PinSocket_1x20_P2.54mm_Vertical"
-			(at 152.4 54.61 0)
-			(effects
-				(font
-					(size 1.27 1.27)
-				)
-				(hide yes)
-			)
-		)
-		(property "Datasheet" "~"
+		(property "Footprint" "MiSTeryShield20kRPiPico:PinSocket_1x20_P2.54mm_Vertical"
 			(at 152.4 54.61 0)
 			(effects
@@
 			)
 		)
-		(property "Description" "Generic connector, single row, 01x20, script generated"
-			(at 152.4 54.61 0)
-			(effects
-				(font
-					(size 1.27 1.27)
-				)
-				(hide yes)
-			)
-		)
-		(property "JLCPCB Position Offset" ""
+		(property "Datasheet" ""
 			(at 152.4 54.61 0)
 			(effects
@@
 			)
 		)
-		(property "JLCPCB Rotation Offset" ""
+		(property "Description" ""
 			(at 152.4 54.61 0)
 			(effects
@@
 			)
 		)
-		(property "Comment" "1x20, P2.54mm"
-			(at 152.4 54.61 0)
-			(effects
-				(font
-					(size 1.27 1.27)
-				)
-				(hide yes)
-			)
-		)
 		(pin "1"
 		)
@@
 	(symbol
 		(lib_id "Connector:Conn_01x02_Pin")
-		(at 255.27 137.16 270)
+		(at 252.73 137.16 90)
+		(mirror x)
 		(unit 1)
 		(exclude_from_sim no)
@@
 		(dnp no)
 		(property "Reference" "J5"
-			(at 249.936 136.652 90)
+			(at 252.222 135.89 90)
 			(effects
 				(font
@@
 		)
 		(property "Value" "Conn_01x02_Pin"
-			(at 256.032 136.906 90)
+			(at 270.256 135.89 90)
 			(effects
 				(font
@@
 			)
 		)
-		(property "Footprint" "Connector_PinHeader_2.54mm:PinHeader_1x02_P2.54mm_Horizontal"
-			(at 255.27 137.16 0)
+		(property "Footprint" "MiSTeryShield20kRPiPico:HDR-TH_2P-P2.54-H-M-W10.4"
+			(at 252.73 137.16 0)
 			(effects
 				(font
@@
 			)
 		)
-		(property "Datasheet" "~"
-			(at 255.27 137.16 0)
+		(property "Datasheet" ""
+			(at 252.73 137.16 0)
 			(effects
 				(font
@@
 			)
 		)
-		(property "Description" "Generic connector, single row, 01x02, script generated"
-			(at 255.27 137.16 0)
+		(property "Description" ""
+			(at 252.73 137.16 0)
 			(effects
 				(font
@@
 		)
 		(property "JLCPCB Part #" "C492410"
-			(at 255.27 137.16 0)
+			(at 252.73 137.16 0)
 			(effects
 				(font
