File: misteryshield20k_rpipico_dual_db9/MiSTeryShield20kRPiPicoUSB_usbhub.kicad_sch (KiCad schematic)
At the start: 17 parts, among them J11 USB_A_Stacked, J12 USB_A_Stacked, J8 Conn_01x20_Pin, J9 Conn_01x20_Pin, U4 CH334U, Y1 Crystal_GND24

Commit message: Add files via upload
Connections:
- net PI_UART_RX: no longer names the net of J8.2 (Pin_2)
- net PI_UART_TX: no longer names the net of J8.1 (Pin_1)
- no-connect marks 26 -> 28
Changed lines of the file:
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@@
+	)
+	(no_connect
+		(at 66.04 36.83)
 	)
 	(no_connect
@@
 	)
 	(no_connect
+		(at 66.04 34.29)
+	)
+	(no_connect
 		(at 198.12 58.42)
 	)
@@
 	(wire
 		(pts
-			(xy 45.72 34.29) (xy 66.04 34.29)
-		)
-		(stroke
-			(width 0)
-			(type default)
-		)
-	)
-	(wire
-		(pts
 			(xy 45.72 44.45) (xy 66.04 44.45)
 		)
@@
 		(pts
 			(xy 250.19 111.76) (xy 250.19 114.3)
-		)
-		(stroke
-			(width 0)
-			(type default)
-		)
-	)
-	(wire
-		(pts
-			(xy 45.72 36.83) (xy 66.04 36.83)
 		)
 		(stroke
@@
 		)
 	)
-	(label "PI_UART_TX"
-		(at 48.26 34.29 0)
-		(effects
-			(font
-				(size 1.27 1.27)
-			)
-			(justify left bottom)
-		)
-	)
 	(label "UP_D-"
 		(at 207.01 68.58 180)
@@
 		(effects
 			(font
-				(size 1.27 1.27)
-			)
-			(justify left bottom)
-		)
-	)
-	(label "PI_UART_RX"
-		(at 48.26 36.83 0)
-		(effects
-			(font

Commit message: Add files via upload
Parts:
- added H5: 2x4 Pinheader horizontal, MiSTeryShield20kRPiPico:HDR-TH_8P-P2.54-H-M-R2-C4-S2.54-N, symbol MiSTeryShield20kRPiPico:PZ254-2-04-W-8.5
Connections:
- net +5V: now also H5.8
- net GND: now also H5.6
- net PI_UART_TX: now reaches J8.1 (Pin_1)
- net PI_UART_TX: now also H5.1
- net PI_UART_RX: now reaches J8.2 (Pin_2)
- net PI_UART_RX: now also H5.2
- new net +3.3V: H5.7
- new net UART_RX: H5.3
- new net UART_TX: H5.4
- no-connect marks 28 -> 27

Commit message: Add files via upload
Parts:
- H5: LCSC Part #  (none) -> C2894984; Supplier Part C2894984 -> (none)
Other:
- note added: "CH334U"
- note added: "Debug Header"
- note added: "PiPico W"
- title: MiSTeryShield20KRPiPico -> MiSTeryShield-20K-PiPico-dual-DB9
- moved on the sheet: H5
Changed lines of the file:
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@@
 	(paper "A4")
 	(title_block
-		(title "MiSTeryShield20KRPiPico")
-		(date "2025-08-09")
-		(rev "V3")
+		(title "MiSTeryShield-20K-PiPico-dual-DB9")
+		(date "2026-01-25")
+		(rev "V1")
 		(company "Stefan Voss")
-		(comment 3 "(c) 2025 by Stefan Voss")
+		(comment 3 "Original Design (c) 2025 by Stefan Voss")
 		(comment 4 "MiSTery Pi Pico WLAN Shield for Tang Nano 20K")
 	)
+	(text "CH334U"
+		(exclude_from_sim no)
+		(at 175.514 23.114 0)
+		(effects
+			(font
+				(size 2.032 2.032)
+			)
+			(justify left bottom)
+		)
+	)
+	(text "PiPico W"
+		(exclude_from_sim no)
+		(at 76.454 23.114 0)
+		(effects
+			(font
+				(size 2.032 2.032)
+			)
+			(justify left bottom)
+		)
+	)
+	(text "Debug Header"
+		(exclude_from_sim no)
+		(at 169.418 90.424 0)
+		(effects
+			(font
+				(size 2.032 2.032)
+			)
+			(justify left bottom)
+		)
+	)
 	(junction
 		(at 250.19 114.3)
@@
 	)
 	(no_connect
-		(at 177.8 101.6)
+		(at 185.42 107.95)
 	)
 	(no_connect
@@
 	(wire
 		(pts
-			(xy 172.72 104.14) (xy 177.8 104.14)
+			(xy 180.34 110.49) (xy 185.42 110.49)
 		)
 		(stroke
@@
 	(wire
 		(pts
-			(xy 193.04 101.6) (xy 187.96 101.6)
+			(xy 200.66 107.95) (xy 195.58 107.95)
 		)
 		(stroke
@@
 	(wire
 		(pts
-			(xy 187.96 96.52) (xy 207.01 96.52)
+			(xy 195.58 102.87) (xy 214.63 102.87)
 		)
 		(stroke
@@
 	(wire
 		(pts
-			(xy 194.31 99.06) (xy 187.96 99.06)
+			(xy 201.93 105.41) (xy 195.58 105.41)
 		)
 		(stroke
@@
 	(wire
 		(pts
-			(xy 157.48 96.52) (xy 177.8 96.52)
+			(xy 165.1 102.87) (xy 185.42 102.87)
 		)
 		(stroke
@@
 	(wire
 		(pts
-			(xy 193.04 104.14) (xy 187.96 104.14)
+			(xy 200.66 110.49) (xy 195.58 110.49)
 		)
 		(stroke
@@
 	(wire
 		(pts
-			(xy 171.45 99.06) (xy 177.8 99.06)
+			(xy 179.07 105.41) (xy 185.42 105.41)
 		)
 		(stroke
@@
 	)
 	(label "PI_UART_TX"
-		(at 160.02 96.52 0)
+		(at 167.64 102.87 0)
 		(effects
 			(font
@@
 	)
 	(label "PI_UART_RX"
-		(at 204.47 96.52 180)
+		(at 212.09 102.87 180)
 		(effects
 			(font
@@
 	(hierarchical_label "UART_TX"
 		(shape output)
-		(at 194.31 99.06 0)
+		(at 201.93 105.41 0)
 		(effects
 			(font
@@
 	(hierarchical_label "UART_RX"
 		(shape input)
-		(at 171.45 99.06 180)
+		(at 179.07 105.41 180)
 		(effects
 			(font
@@
 	(symbol
 		(lib_id "power:GND")
-		(at 193.04 101.6 90)
+		(at 200.66 107.95 90)
 		(mirror x)
 		(unit 1)
@@
 		(dnp no)
 		(property "Reference" "#PWR042"
-			(at 199.39 101.6 0)
+			(at 207.01 107.95 0)
 			(effects
 				(font
@@
 		)
 		(property "Value" "GND"
-			(at 196.85 101.6 90)
+			(at 204.47 107.95 90)
 			(effects
 				(font
@@
 		)
 		(property "Footprint" ""
-			(at 193.04 101.6 0)
+			(at 200.66 107.95 0)
 			(effects
 				(font
@@
 		)
 		(property "Datasheet" ""
-			(at 193.04 101.6 0)
+			(at 200.66 107.95 0)
 			(effects
 				(font
@@
 		)
 		(property "Description" ""
-			(at 193.04 101.6 0)
+			(at 200.66 107.95 0)
 			(effects
 				(font
@@
 	(symbol
 		(lib_id "MiSTeryShield20kRPiPico:PZ254-2-04-W-8.5")
-		(at 182.88 100.33 0)
+		(at 190.5 106.68 0)
 		(unit 1)
 		(exclude_from_sim no)
@@
 		(fields_autoplaced yes)
 		(property "Reference" "H5"
-			(at 182.88 88.9 0)
+			(at 190.5 95.25 0)
 			(effects
 				(font
@@
 		)
 		(property "Value" "2x4 Pinheader horizontal"
-			(at 182.88 91.44 0)
+			(at 190.5 97.79 0)
 			(effects
 				(font
@@
 		)
 		(property "Footprint" "MiSTeryShield20kRPiPico:HDR-TH_8P-P2.54-H-M-R2-C4-S2.54-N"
-			(at 182.88 100.33 0)
+			(at 190.5 106.68 0)
 			(effects
 				(font
@@
 		)
 		(property "Datasheet" "https://item.szlcsc.com/datasheet/PZ254-2-04-W-8.5/3132660.html"
-			(at 182.88 100.33 0)
+			(at 190.5 106.68 0)
 			(effects
 				(font
@@
 		)
 		(property "Description" "Pin Structure:2x4P Pitch:2.54mm Row Spacing:2.54mm Circluar Pins/Square Pins:Pin Header Mounting Type:Right Angle Number of Rows:2 Number of Pins:8P Current Rating:3A Voltage Rating (Max):- Length of Mating Pin:6mm Insulation Height:2.5mm Length of End Co"
-			(at 182.88 100.33 0)
+			(at 190.5 106.68 0)
 			(effects
 				(font
@@
 		)
 		(property "Manufacturer Part" "PZ254-2-04-W-8.5"
-			(at 182.88 100.33 0)
+			(at 190.5 106.68 0)
 			(effects
 				(font
@@
 		)
 		(property "Manufacturer" "HCTL(华灿天禄)"
-			(at 182.88 100.33 0)
+			(at 190.5 106.68 0)
 			(effects
 				(font
@@
 			)
 		)
-		(property "Supplier Part" "C2894984"
-			(at 182.88 100.33 0)
+		(property "Supplier" "LCSC"
+			(at 190.5 106.68 0)
 			(effects
 				(font
@@
 			)
 		)
-		(property "Supplier" "LCSC"
-			(at 182.88 100.33 0)
+		(property "LCSC Part Name" "2x4P 间距:2.54mm 方针 弯插"
+			(at 190.5 106.68 0)
 			(effects
 				(font
@@
 			)
 		)
-		(property "LCSC Part Name" "2x4P 间距:2.54mm 方针 弯插"
-			(at 182.88 100.33 0)
+		(property "LCSC Part # " "C2894984"
+			(at 190.5 106.68 0)
 			(effects
 				(font
@@
 	(symbol
 		(lib_id "power:+5V")
-		(at 193.04 104.14 270)
+		(at 200.66 110.49 270)
 		(mirror x)
 		(unit 1)
@@
 		(dnp no)
 		(property "Reference" "#PWR0101"
-			(at 189.23 104.14 0)
+			(at 196.85 110.49 0)
 			(effects
 				(font
@@
 		)
 		(property "Value" "+5V"
-			(at 196.85 104.14 90)
+			(at 204.47 110.49 90)
 			(effects
 				(font
@@
 		)
 		(property "Footprint" ""
-			(at 193.04 104.14 0)
+			(at 200.66 110.49 0)
 			(effects
 				(font
@@
 		)
 		(property "Datasheet" ""
-			(at 193.04 104.14 0)
+			(at 200.66 110.49 0)
 			(effects
 				(font
@@
 		)
 		(property "Description" ""
-			(at 193.04 104.14 0)
+			(at 200.66 110.49 0)
 			(effects
 				(font
@@
 	(symbol
 		(lib_id "power:+3.3V")
-		(at 172.72 104.14 90)
+		(at 180.34 110.49 90)
 		(mirror x)
 		(unit 1)
@@
 		(dnp no)
 		(property "Reference" "#PWR043"
-			(at 176.53 104.14 0)
+			(at 184.15 110.49 0)
 			(effects
 				(font
@@
 		)
 		(property "Value" "+3.3V"
-			(at 169.545 104.14 90)
+			(at 177.165 110.49 90)
 			(effects
 				(font
@@
 		)
 		(property "Footprint" ""
-			(at 172.72 104.14 0)
+			(at 180.34 110.49 0)
 			(effects
 				(font
@@
 		)
 		(property "Datasheet" ""
-			(at 172.72 104.14 0)
+			(at 180.34 110.49 0)
 			(effects
 				(font
@@
 		)
 		(property "Description" ""
-			(at 172.72 104.14 0)
+			(at 180.34 110.49 0)
 			(effects
 				(font

Commit message: Add files via upload
Parts:
- H5: value 2x4 Pinheader horizontal -> 2x3 Pinheader horizontal; footprint MiSTeryShield20kRPiPico:HDR-TH_8P-P2.54-H-M-R2-C4-S2.54-N -> Connector_PinHeader_2.54mm:PinHeader_2x03_P2.54mm_Horizontal; symbol MiSTeryShield20kRPiPico:PZ254-2-04-W-8.5 -> Connector_Generic:Conn_02x03_Odd_Even; Supplier Part (none) -> C2894984
Connections:
- net +5V: no longer H5.8
- net GND: now also H5.1 (Pin_1), H5.2 (Pin_2); no longer H5.6
- net PI_UART_RX: now also H5.5 (Pin_5); no longer H5.2
- net PI_UART_TX: now also H5.6 (Pin_6); no longer H5.1
- removed net +3.3V: H5.7
- no-connect marks 27 -> 26

Commit message: Add files via upload
Parts:
- D2, D3, D4: value green -> orange; LCSC Part # C2297 -> C110371
Other:
- moved on the sheet: D3, D4, R19, R20
Changed lines of the file:
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@@
 	(wire
 		(pts
-			(xy 35.56 49.53) (xy 35.56 55.88)
+			(xy 38.1 49.53) (xy 38.1 55.88)
 		)
 		(stroke
@@
 	(wire
 		(pts
-			(xy 66.04 49.53) (xy 35.56 49.53)
+			(xy 66.04 49.53) (xy 38.1 49.53)
 		)
 		(stroke
@@
 	(wire
 		(pts
-			(xy 66.04 54.61) (xy 44.45 54.61)
+			(xy 66.04 54.61) (xy 49.53 54.61)
 		)
 		(stroke
@@
 	(wire
 		(pts
-			(xy 44.45 54.61) (xy 44.45 55.88)
+			(xy 49.53 54.61) (xy 49.53 55.88)
 		)
 		(stroke
@@
 			)
 		)
-		(property "Value" "green"
+		(property "Value" "orange"
 			(at 30.48 62.5474 90)
 			(effects
@@
 			)
 		)
-		(property "LCSC Part #" "C2297"
+		(property "LCSC Part #" " C110371"
 			(at 26.67 59.69 0)
 			(effects
@@
 	(symbol
 		(lib_id "Device:LED")
-		(at 35.56 59.69 90)
+		(at 38.1 59.69 90)
 		(unit 1)
 		(exclude_from_sim no)
@@
 		(fields_autoplaced yes)
 		(property "Reference" "D3"
-			(at 39.37 60.0074 90)
+			(at 41.91 60.0074 90)
 			(effects
 				(font
@@
 			)
 		)
-		(property "Value" "green"
-			(at 39.37 62.5474 90)
+		(property "Value" "orange"
+			(at 41.91 62.5474 90)
 			(effects
 				(font
@@
 		)
 		(property "Footprint" "LED_SMD:LED_0805_2012Metric"
-			(at 35.56 59.69 0)
+			(at 38.1 59.69 0)
 			(effects
 				(font
@@
 		)
 		(property "Datasheet" "~"
-			(at 35.56 59.69 0)
+			(at 38.1 59.69 0)
 			(effects
 				(font
@@
 		)
 		(property "Description" ""
-			(at 35.56 59.69 0)
+			(at 38.1 59.69 0)
 			(effects
 				(font
@@
 			)
 		)
-		(property "LCSC Part #" "C2297"
-			(at 35.56 59.69 0)
+		(property "LCSC Part #" " C110371"
+			(at 38.1 59.69 0)
 			(effects
 				(font
@@
 		)
 		(property "JLCPCB Position Offset" ""
-			(at 35.56 59.69 0)
+			(at 38.1 59.69 0)
 			(effects
 				(font
@@
 		)
 		(property "JLCPCB Rotation Offset" ""
-			(at 35.56 59.69 0)
+			(at 38.1 59.69 0)
 			(effects
 				(font
@@
 		)
 		(property "Comment" "0805"
-			(at 35.56 59.69 0)
+			(at 38.1 59.69 0)
 			(effects
 				(font
@@
 	(symbol
 		(lib_id "power:GND")
-		(at 35.56 71.12 0)
+		(at 38.1 71.12 0)
 		(unit 1)
 		(exclude_from_sim no)
@@
 		(fields_autoplaced yes)
 		(property "Reference" "#PWR058"
-			(at 35.56 77.47 0)
+			(at 38.1 77.47 0)
 			(effects
 				(font
@@
 		)
 		(property "Value" "GND"
-			(at 35.56 76.454 0)
+			(at 38.1 76.454 0)
 			(effects
 				(font
@@
 		)
 		(property "Footprint" ""
-			(at 35.56 71.12 0)
+			(at 38.1 71.12 0)
 			(effects
 				(font
@@
 		)
 		(property "Datasheet" ""
-			(at 35.56 71.12 0)
+			(at 38.1 71.12 0)
 			(effects
 				(font
@@
 		)
 		(property "Description" ""
-			(at 35.56 71.12 0)
+			(at 38.1 71.12 0)
 			(effects
 				(font
@@
 	(symbol
 		(lib_id "Device:R")
-		(at 35.56 67.31 0)
+		(at 38.1 67.31 0)
 		(unit 1)
 		(exclude_from_sim no)
@@
 		(fields_autoplaced yes)
 		(property "Reference" "R19"
-			(at 38.1 66.0399 0)
+			(at 40.64 66.0399 0)
 			(effects
 				(font
@@
 		)
 		(property "Value" "560"
-			(at 38.1 68.5799 0)
+			(at 40.64 68.5799 0)
 			(effects
 				(font
@@
 		)
 		(property "Footprint" "Resistor_SMD:R_0805_2012Metric"
-			(at 33.782 67.31 90)
+			(at 36.322 67.31 90)
 			(effects
 				(font
@@
 		)
 		(property "Datasheet" "~"
-			(at 35.56 67.31 0)
+			(at 38.1 67.31 0)
 			(effects
 				(font
@@
 		)
 		(property "Description" ""
-			(at 35.56 67.31 0)
+			(at 38.1 67.31 0)
 			(effects
 				(font
@@
 		)
 		(property "LCSC Part #" "C28636"
-			(at 35.56 67.31 0)
+			(at 38.1 67.31 0)
 			(effects
 				(font
@@
 		)
 		(property "JLCPCB Position Offset" ""
-			(at 35.56 67.31 0)
+			(at 38.1 67.31 0)
 			(effects
 				(font
@@
 		)
 		(property "JLCPCB Rotation Offset" ""
-			(at 35.56 67.31 0)
+			(at 38.1 67.31 0)
 			(effects
 				(font
@@
 		)
 		(property "Comment" "0805"
-			(at 35.56 67.31 0)
+			(at 38.1 67.31 0)
 			(effects
 				(font
@@
 	(symbol
 		(lib_id "power:GND")
-		(at 44.45 71.12 0)
+		(at 49.53 71.12 0)
 		(unit 1)
 		(exclude_from_sim no)
@@
 		(fields_autoplaced yes)
 		(property "Reference" "#PWR059"
-			(at 44.45 77.47 0)
+			(at 49.53 77.47 0)
 			(effects
 				(font
@@
 		)
 		(property "Value" "GND"
-			(at 44.45 76.454 0)
+			(at 49.53 76.454 0)
 			(effects
 				(font
@@
 		)
 		(property "Footprint" ""
-			(at 44.45 71.12 0)
+			(at 49.53 71.12 0)
 			(effects
 				(font
@@
 		)
 		(property "Datasheet" ""
-			(at 44.45 71.12 0)
+			(at 49.53 71.12 0)
 			(effects
 				(font
@@
 		)
 		(property "Description" ""
-			(at 44.45 71.12 0)
+			(at 49.53 71.12 0)
 			(effects
 				(font
@@
 	(symbol
 		(lib_id "Device:R")
-		(at 44.45 67.31 0)
+		(at 49.53 67.31 0)
 		(unit 1)
 		(exclude_from_sim no)
@@
 		(fields_autoplaced yes)
 		(property "Reference" "R20"
-			(at 46.99 66.0399 0)
+			(at 52.07 66.0399 0)
 			(effects
 				(font
@@
 		)
 		(property "Value" "560"
-			(at 46.99 68.5799 0)
+			(at 52.07 68.5799 0)
 			(effects
 				(font
@@
 		)
 		(property "Footprint" "Resistor_SMD:R_0805_2012Metric"
-			(at 42.672 67.31 90)
+			(at 47.752 67.31 90)
 			(effects
 				(font
@@
 		)
 		(property "Datasheet" "~"
-			(at 44.45 67.31 0)
+			(at 49.53 67.31 0)
 			(effects
 				(font
@@
 		)
 		(property "Description" ""
-			(at 44.45 67.31 0)
+			(at 49.53 67.31 0)
 			(effects
 				(font
@@
 		)
 		(property "LCSC Part #" "C28636"
-			(at 44.45 67.31 0)
+			(at 49.53 67.31 0)
 			(effects
 				(font
@@
 		)
 		(property "JLCPCB Position Offset" ""
-			(at 44.45 67.31 0)
+			(at 49.53 67.31 0)
 			(effects
 				(font
@@
 		)
 		(property "JLCPCB Rotation Offset" ""
-			(at 44.45 67.31 0)
+			(at 49.53 67.31 0)
 			(effects
 				(font
@@
 		)
 		(property "Comment" "0805"
-			(at 44.45 67.31 0)
+			(at 49.53 67.31 0)
 			(effects
 				(font
@@
 	(symbol
 		(lib_id "Device:LED")
-		(at 44.45 59.69 90)
+		(at 49.53 59.69 90)
 		(unit 1)
 		(exclude_from_sim no)
@@
 		(fields_autoplaced yes)
 		(property "Reference" "D4"
-			(at 48.26 60.0074 90)
+			(at 53.34 60.0074 90)
 			(effects
 				(font
@@
 			)
 		)
-		(property "Value" "green"
-			(at 48.26 62.5474 90)
+		(property "Value" "orange"
+			(at 53.34 62.5474 90)
 			(effects
 				(font
@@
 		)
 		(property "Footprint" "LED_SMD:LED_0805_2012Metric"
-			(at 44.45 59.69 0)
+			(at 49.53 59.69 0)
 			(effects
 				(font
@@
 		)
 		(property "Datasheet" "~"
-			(at 44.45 59.69 0)
+			(at 49.53 59.69 0)
 			(effects
 				(font
@@
 		)
 		(property "Description" ""
-			(at 44.45 59.69 0)
+			(at 49.53 59.69 0)
 			(effects
 				(font
@@
 			)
 		)
-		(property "LCSC Part #" "C2297"
-			(at 44.45 59.69 0)
+		(property "LCSC Part #" " C110371"
+			(at 49.53 59.69 0)
 			(effects
 				(font
@@
 		)
 		(property "JLCPCB Position Offset" ""
-			(at 44.45 59.69 0)
+			(at 49.53 59.69 0)
 			(effects
 				(font
@@
 		)
 		(property "JLCPCB Rotation Offset" ""
-			(at 44.45 59.69 0)
+			(at 49.53 59.69 0)
 			(effects
 				(font
@@
 		)
 		(property "Comment" "0805"
-			(at 44.45 59.69 0)
+			(at 49.53 59.69 0)
 			(effects
 				(font

Commit message: Add files via upload
Parts:
- D2, D3, D4: footprint LED_SMD:LED_0805_2012Metric -> MiSTeryShield20kRPiPico:LED0805-RD; JLC_3DModel_Q (none) -> 23093642268545519703b953fc993978; JLC_3D_Size (none) -> 2.02 1.25
Changed lines of the file:
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@@
 			)
 		)
-		(property "Footprint" "LED_SMD:LED_0805_2012Metric"
+		(property "Footprint" "MiSTeryShield20kRPiPico:LED0805-RD"
 			(at 26.67 59.69 0)
 			(effects
@@
 			)
 		)
-		(property "Datasheet" "~"
+		(property "Datasheet" ""
 			(at 26.67 59.69 0)
 			(effects
@@
 		)
 		(property "Comment" "0805"
+			(at 26.67 59.69 0)
+			(effects
+				(font
+					(size 1.27 1.27)
+				)
+				(hide yes)
+			)
+		)
+		(property "JLC_3DModel_Q" "23093642268545519703b953fc993978"
+			(at 26.67 59.69 0)
+			(effects
+				(font
+					(size 1.27 1.27)
+				)
+				(hide yes)
+			)
+		)
+		(property "JLC_3D_Size" "2.02 1.25"
 			(at 26.67 59.69 0)
 			(effects
@@
 			)
 		)
-		(property "Footprint" "LED_SMD:LED_0805_2012Metric"
+		(property "Footprint" "MiSTeryShield20kRPiPico:LED0805-RD"
 			(at 38.1 59.69 0)
 			(effects
@@
 			)
 		)
-		(property "Datasheet" "~"
+		(property "Datasheet" ""
 			(at 38.1 59.69 0)
 			(effects
@@
 		)
 		(property "Comment" "0805"
+			(at 38.1 59.69 0)
+			(effects
+				(font
+					(size 1.27 1.27)
+				)
+				(hide yes)
+			)
+		)
+		(property "JLC_3DModel_Q" "23093642268545519703b953fc993978"
+			(at 38.1 59.69 0)
+			(effects
+				(font
+					(size 1.27 1.27)
+				)
+				(hide yes)
+			)
+		)
+		(property "JLC_3D_Size" "2.02 1.25"
 			(at 38.1 59.69 0)
 			(effects
@@
 			)
 		)
-		(property "Footprint" "LED_SMD:LED_0805_2012Metric"
+		(property "Footprint" "MiSTeryShield20kRPiPico:LED0805-RD"
 			(at 49.53 59.69 0)
 			(effects
@@
 			)
 		)
-		(property "Datasheet" "~"
+		(property "Datasheet" ""
 			(at 49.53 59.69 0)
 			(effects
@@
 			(at 49.53 59.69 0)
 			(effects
+				(font
+					(size 1.27 1.27)
+				)
+				(hide yes)
+			)
+		)
+		(property "JLC_3DModel_Q" "23093642268545519703b953fc993978"
+			(at 49.53 59.69 0)
+			(effects
+				(font
+					(size 1.27 1.27)
+				)
+				(hide yes)
+			)
+		)
+		(property "JLC_3D_Size" "2.02 1.25"
+			(at 49.53 59.69 0)
+			(effects

Commit message: Add files via upload
Parts:
- D2, D3, D4: LCSC (none) -> C110371
- H5: JLCPCB Rotation Offset (none) -> 90; Supplier Part C2894984 -> (none)
- R18, R19, R20: value 560 -> 510; LCSC Part # C28636 -> C17734
Changed lines of the file:
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@@
 			)
 		)
-		(property "Value" "560"
+		(property "Value" "510"
 			(at 29.21 68.5799 0)
 			(effects
@@
 			)
 		)
-		(property "LCSC Part #" "C28636"
+		(property "LCSC Part #" "C17734"
 			(at 26.67 67.31 0)
 			(effects
@@
 			)
 		)
+		(property "LCSC" "C110371"
+			(at 26.67 59.69 0)
+			(effects
+				(font
+					(size 1.27 1.27)
+				)
+				(hide yes)
+			)
+		)
 		(pin "2"
 		)
@@
 		)
 		(property "JLC_3D_Size" "2.02 1.25"
+			(at 38.1 59.69 0)
+			(effects
+				(font
+					(size 1.27 1.27)
+				)
+				(hide yes)
+			)
+		)
+		(property "LCSC" "C110371"
 			(at 38.1 59.69 0)
 			(effects
@@
 			)
 		)
-		(property "Supplier Part" "C2894984"
+		(property "JLCPCB Rotation Offset" "90"
 			(at 190.5 105.41 0)
 			(effects
@@
 			)
 		)
-		(property "Value" "560"
+		(property "Value" "510"
 			(at 40.64 68.5799 0)
 			(effects
@@
 			)
 		)
-		(property "LCSC Part #" "C28636"
+		(property "LCSC Part #" "C17734"
 			(at 38.1 67.31 0)
 			(effects
@@
 			)
 		)
-		(property "Value" "560"
+		(property "Value" "510"
 			(at 52.07 68.5799 0)
 			(effects
@@
 			)
 		)
-		(property "LCSC Part #" "C28636"
+		(property "LCSC Part #" "C17734"
 			(at 49.53 67.31 0)
 			(effects
@@
 			(at 49.53 59.69 0)
 			(effects
+				(font
+					(size 1.27 1.27)
+				)
+				(hide yes)
+			)
+		)
+		(property "LCSC" "C110371"
+			(at 49.53 59.69 0)
+			(effects
