File: misteryshield20k_rpipico_dual_db9/MiSTeryShield20kRPiPicoUSB_usbhub.kicad_sch (KiCad schematic)
At the start: 18 parts, among them J11 USB_A_Stacked, J12 USB_A_Stacked, J8 Conn_01x20_Pin, J9 Conn_01x20_Pin, U4 CH334U, Y1 Crystal_GND24

Commit message: Add files via upload
Parts:
- H5: footprint Connector_PinHeader_2.54mm:PinHeader_2x03_P2.54mm_Horizontal -> MiSTeryShield20kRPiPico:HDR-TH_6P-P2.54-H-M-R2-C3-S2.54-W12.3-N; JLCPCB Rotation Offset 90 -> 0; LCSC Part # (none) -> C2894983; LCSC Part #  C2894984 -> (none); LCSC Part Name 2x4P 间距:2.54mm 方针 弯插 -> (none); Manufacturer Part PZ254-2-04-W-8.5 -> PZ254-2-03-W-8.5
- J8: footprint Connector_PinSocket_2.54mm:PinSocket_1x20_P2.54mm_Vertical -> MiSTeryShield20kRPiPico:PinSocket_1x20_P2.54mm_Vertical
- J9: footprint Connector_PinSocket_2.54mm:PinSocket_1x20_P2.54mm_Vertical -> MiSTeryShield20kRPiPico:PinSocket_1x20_P2.54mm_Vertical; JLCPCB Rotation Offset (none) -> 90
Connections:
- net GND: now also H5.5 (Pin_5), H5.6 (Pin_6); no longer H5.1 (Pin_1), H5.2 (Pin_2)
- net PI_UART_RX: now also H5.2 (Pin_2); no longer H5.5 (Pin_5)
- net PI_UART_TX: now also H5.1 (Pin_1); no longer H5.6 (Pin_6)
- net UART_RX: now also H5.4 (Pin_4); no longer H5.3 (Pin_3)
- net UART_TX: now also H5.3 (Pin_3); no longer H5.4 (Pin_4)
Changed lines of the file:
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@@
 	(wire
 		(pts
-			(xy 205.74 53.34) (xy 205.74 57.15)
+			(xy 171.45 102.87) (xy 185.42 102.87)
 		)
 		(stroke
@@
 	(wire
 		(pts
-			(xy 66.04 49.53) (xy 38.1 49.53)
+			(xy 180.34 107.95) (xy 185.42 107.95)
 		)
 		(stroke
@@
 	(wire
 		(pts
-			(xy 218.44 54.61) (xy 218.44 55.88)
+			(xy 205.74 53.34) (xy 205.74 57.15)
 		)
 		(stroke
@@
 	(wire
 		(pts
-			(xy 127 69.85) (xy 133.35 69.85)
+			(xy 66.04 49.53) (xy 38.1 49.53)
 		)
 		(stroke
@@
 	(wire
 		(pts
-			(xy 205.74 62.23) (xy 205.74 63.5)
+			(xy 218.44 54.61) (xy 218.44 55.88)
 		)
 		(stroke
@@
 	(wire
 		(pts
-			(xy 63.5 52.07) (xy 66.04 52.07)
+			(xy 127 69.85) (xy 133.35 69.85)
 		)
 		(stroke
@@
 	(wire
 		(pts
-			(xy 246.38 68.58) (xy 246.38 69.85)
+			(xy 205.74 62.23) (xy 205.74 63.5)
 		)
 		(stroke
@@
 	(wire
 		(pts
-			(xy 198.12 107.95) (xy 218.44 107.95)
+			(xy 63.5 52.07) (xy 66.04 52.07)
+		)
+		(stroke
+			(width 0)
+			(type default)
+		)
+	)
+	(wire
+		(pts
+			(xy 246.38 68.58) (xy 246.38 69.85)
 		)
 		(stroke
@@
 	(wire
 		(pts
-			(xy 203.2 102.87) (xy 198.12 102.87)
-		)
-		(stroke
-			(width 0)
-			(type default)
-		)
-	)
-	(wire
-		(pts
 			(xy 127 74.93) (xy 133.35 74.93)
 		)
@@
 	(wire
 		(pts
-			(xy 180.34 102.87) (xy 185.42 102.87)
-		)
-		(stroke
-			(width 0)
-			(type default)
-		)
-	)
-	(wire
-		(pts
 			(xy 45.72 36.83) (xy 66.04 36.83)
 		)
@@
 	(wire
 		(pts
+			(xy 200.66 105.41) (xy 198.12 105.41)
+		)
+		(stroke
+			(width 0)
+			(type default)
+		)
+	)
+	(wire
+		(pts
 			(xy 127 64.77) (xy 129.54 64.77)
 		)
@@
 	(wire
 		(pts
+			(xy 203.2 107.95) (xy 198.12 107.95)
+		)
+		(stroke
+			(width 0)
+			(type default)
+		)
+	)
+	(wire
+		(pts
 			(xy 269.24 85.09) (xy 269.24 86.36)
 		)
@@
 	(wire
 		(pts
+			(xy 198.12 102.87) (xy 217.17 102.87)
+		)
+		(stroke
+			(width 0)
+			(type default)
+		)
+	)
+	(wire
+		(pts
 			(xy 158.75 63.5) (xy 172.72 63.5)
 		)
@@
 	(wire
 		(pts
-			(xy 166.37 107.95) (xy 185.42 107.95)
+			(xy 181.61 105.41) (xy 185.42 105.41)
 		)
 		(stroke
@@
 	(wire
 		(pts
-			(xy 170.18 105.41) (xy 185.42 105.41)
-		)
-		(stroke
-			(width 0)
-			(type default)
-		)
-	)
-	(wire
-		(pts
 			(xy 207.01 66.04) (xy 198.12 66.04)
 		)
@@
 	(wire
 		(pts
-			(xy 212.09 105.41) (xy 198.12 105.41)
-		)
-		(stroke
-			(width 0)
-			(type default)
-		)
-	)
-	(wire
-		(pts
 			(xy 66.04 39.37) (xy 63.5 39.37)
 		)
@@
 	)
 	(label "PI_UART_TX"
-		(at 199.39 107.95 0)
+		(at 172.72 102.87 0)
 		(effects
 			(font
@@
 		)
 	)
-	(label "USB1_D+"
-		(at 273.05 48.26 180)
+	(label "PI_UART_RX"
+		(at 199.39 102.87 0)
 		(effects
 			(font
 				(size 1.27 1.27)
 			)
-			(justify right bottom)
+			(justify left bottom)
 		)
 	)
-	(label "PI_UART_RX"
-		(at 173.99 107.95 0)
+	(label "USB1_D+"
+		(at 273.05 48.26 180)
 		(effects
 			(font
 				(size 1.27 1.27)
 			)
-			(justify left bottom)
+			(justify right bottom)
 		)
 	)
@@
 	(hierarchical_label "UART_TX"
 		(shape output)
-		(at 212.09 105.41 0)
+		(at 181.61 105.41 180)
 		(effects
 			(font
 				(size 1.27 1.27)
 			)
-			(justify left)
+			(justify right)
 		)
 	)
@@
 		)
 	)
-	(hierarchical_label "RECONFGN"
-		(shape output)
-		(at 133.35 69.85 0)
+	(hierarchical_label "UART_RX"
+		(shape input)
+		(at 200.66 105.41 0)
 		(effects
 			(font
@@
 		)
 	)
-	(hierarchical_label "UART_RX"
-		(shape input)
-		(at 170.18 105.41 180)
+	(hierarchical_label "RECONFGN"
+		(shape output)
+		(at 133.35 69.85 0)
 		(effects
 			(font
 				(size 1.27 1.27)
 			)
-			(justify right)
+			(justify left)
 		)
 	)
@@
 	(symbol
 		(lib_id "power:GND")
-		(at 203.2 102.87 90)
+		(at 180.34 107.95 270)
 		(mirror x)
 		(unit 1)
@@
 		(dnp no)
 		(property "Reference" "#PWR042"
-			(at 209.55 102.87 0)
+			(at 173.99 107.95 0)
 			(effects
 				(font
@@
 		)
 		(property "Value" "GND"
-			(at 207.01 102.87 90)
+			(at 176.53 107.95 90)
 			(effects
 				(font
@@
 		)
 		(property "Footprint" ""
-			(at 203.2 102.87 0)
+			(at 180.34 107.95 0)
 			(effects
 				(font
@@
 		)
 		(property "Datasheet" ""
-			(at 203.2 102.87 0)
+			(at 180.34 107.95 0)
 			(effects
 				(font
@@
 		)
 		(property "Description" ""
-			(at 203.2 102.87 0)
+			(at 180.34 107.95 0)
 			(effects
 				(font
@@
 			)
 		)
-		(property "Footprint" "Connector_PinSocket_2.54mm:PinSocket_1x20_P2.54mm_Vertical"
+		(property "Footprint" "MiSTeryShield20kRPiPico:PinSocket_1x20_P2.54mm_Vertical"
 			(at 71.12 57.15 0)
 			(effects
@@
 			)
 		)
-		(property "Datasheet" "~"
+		(property "Datasheet" ""
 			(at 71.12 57.15 0)
 			(effects
@@
 			)
 		)
-		(property "Description" "Generic connector, single row, 01x20, script generated"
+		(property "Description" ""
 			(at 71.12 57.15 0)
 			(effects
@@
 	(symbol
 		(lib_id "power:GND")
-		(at 180.34 102.87 270)
+		(at 203.2 107.95 90)
 		(mirror x)
 		(unit 1)
@@
 		(dnp no)
 		(property "Reference" "#PWR043"
-			(at 173.99 102.87 0)
+			(at 209.55 107.95 0)
 			(effects
 				(font
@@
 		)
 		(property "Value" "GND"
-			(at 176.53 102.87 90)
+			(at 207.01 107.95 90)
 			(effects
 				(font
@@
 		)
 		(property "Footprint" ""
-			(at 180.34 102.87 0)
+			(at 203.2 107.95 0)
 			(effects
 				(font
@@
 		)
 		(property "Datasheet" ""
-			(at 180.34 102.87 0)
+			(at 203.2 107.95 0)
 			(effects
 				(font
@@
 		)
 		(property "Description" ""
-			(at 180.34 102.87 0)
+			(at 203.2 107.95 0)
 			(effects
 				(font
@@
 			)
 		)
-		(property "Footprint" "Connector_PinHeader_2.54mm:PinHeader_2x03_P2.54mm_Horizontal"
+		(property "Footprint" "MiSTeryShield20kRPiPico:HDR-TH_6P-P2.54-H-M-R2-C3-S2.54-W12.3-N"
 			(at 190.5 105.41 0)
 			(effects
@@
 			)
 		)
-		(property "Datasheet" "~"
+		(property "Datasheet" ""
 			(at 190.5 105.41 0)
 			(effects
@@
 			)
 		)
-		(property "Description" "Generic connector, double row, 02x03, odd/even pin numbering scheme (row 1 odd numbers, row 2 even numbers), script generated (kicad-library-utils/schlib/autogen/connector/)"
+		(property "Description" ""
 			(at 190.5 105.41 0)
 			(effects
@@
 			)
 		)
-		(property "Manufacturer Part" "PZ254-2-04-W-8.5"
+		(property "Manufacturer Part" "PZ254-2-03-W-8.5"
 			(at 190.5 105.41 0)
 			(effects
@@
 			)
 		)
-		(property "LCSC Part Name" "2x4P 间距:2.54mm 方针 弯插"
+		(property "JLCPCB Rotation Offset" "0"
 			(at 190.5 105.41 0)
 			(effects
@@
 			)
 		)
-		(property "LCSC Part # " "C2894984"
-			(at 190.5 105.41 0)
-			(effects
-				(font
-					(size 1.27 1.27)
-				)
-				(hide yes)
-			)
-		)
-		(property "JLCPCB Rotation Offset" "90"
+		(property "LCSC Part #" "C2894983"
 			(at 190.5 105.41 0)
 			(effects
@@
 			)
 		)
-		(property "Footprint" "Connector_PinSocket_2.54mm:PinSocket_1x20_P2.54mm_Vertical"
+		(property "Footprint" "MiSTeryShield20kRPiPico:PinSocket_1x20_P2.54mm_Vertical"
 			(at 121.92 57.15 0)
 			(effects
@@
 			)
 		)
-		(property "Datasheet" "~"
+		(property "Datasheet" ""
 			(at 121.92 57.15 0)
 			(effects
@@
 			)
 		)
-		(property "Description" "Generic connector, single row, 01x20, script generated"
+		(property "Description" ""
 			(at 121.92 57.15 0)
 			(effects
@@
 			)
 		)
-		(property "JLCPCB Rotation Offset" ""
+		(property "JLCPCB Rotation Offset" "90"
 			(at 121.92 57.15 0)
 			(effects
