File: misteryshield20k_rpipico_dual_db9/misteryshield20k_rpipico_dual_db9-rounded.kicad_pcb (KiCad board)
At the start: 2 copper layers, 100 x 57 mm, 78 parts, among them J1 Joystick, J11 USB_A_Stacked, J12 USB_A_Stacked, J2 Joystick, J4 Conn_01x20_Pin, J5 Conn_01x02_Pin, J6 S4B-PH-K-S_LF__SN (Grove 1125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, J7 Conn_01x20_Pin, J8 Conn_01x20_Pin, J9 Conn_01x20_Pin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

Commit message: Add files via upload
Parts:
- D1: footprint MiSTeryShield20kRPiPico:SOD-128_L3.7-W2.5-LS4.7-RD -> MiSTeryShield20kRPiPico:SOD-123_L2.7-W1.6-LS3.7-RD
- H5: footprint Connector_PinHeader_2.54mm:PinHeader_2x03_P2.54mm_Horizontal -> MiSTeryShield20kRPiPico:HDR-TH_6P-P2.54-H-M-R2-C3-S2.54-W12.3-N
- J1, J2: value Joystick -> D-DMR009PM-D002
- J4, J7, J8, J9: footprint Connector_PinSocket_2.54mm:PinSocket_1x20_P2.54mm_Vertical -> MiSTeryShield20kRPiPico:PinSocket_1x20_P2.54mm_Vertical
- J5: footprint Connector_PinHeader_2.54mm:PinHeader_1x02_P2.54mm_Horizontal -> MiSTeryShield20kRPiPico:HDR-TH_2P-P2.54-H-M-W10.4
- J6: value S4B-PH-K-S_LF__SN (Grove 1125S-4P) -> Grove 1125S-4P
- moved H5 2.85 mm to (123.4, 50.7), turned to 180 degrees
- moved J5 1.15 mm to (100.9, 51.8), turned to 0 degrees
- moved D1 0.78 mm to (101.6, 48.3)
- moved R28 0.10 mm to (93.0, 43.0)
- moved R29 0.10 mm to (105.4, 43.0)
- moved U1 0.10 mm to (99.2, 43.3)
- turned J4 to -90 degrees
- turned J7 to -90 degrees
- turned J8 to -90 degrees
- turned J9 to -90 degrees
Connections:
- C10 pad 1: Net-(J5-Pin_2) -> Net-(J5-Pin_1)
- C11 pad 1: Net-(J5-Pin_2) -> Net-(J5-Pin_1)
- F1 pad 2: Net-(J5-Pin_2) -> Net-(J5-Pin_1)
- H5 pad 1: GND -> /Pi_Pico_USB_Hub/PI_UART_TX
- H5 pad 2: GND -> /Pi_Pico_USB_Hub/PI_UART_RX
- H5 pad 3: P75 -> /UART_TX
- H5 pad 4: /UART_TX -> P75
- H5 pad 5: /Pi_Pico_USB_Hub/PI_UART_RX -> GND
- H5 pad 6: /Pi_Pico_USB_Hub/PI_UART_TX -> GND
- J5 pad 1: +5V -> Net-(J5-Pin_1)
- J5 pad 2: Net-(J5-Pin_2) -> +5V
Routing:
- net Net-(J5-Pin_1): track 0.00 -> 8.52 mm
- net Net-(J5-Pin_2): track 8.40 -> 0.00 mm
- net Net-(D1-K): track 11.8 -> 14.0 mm
- net P77: track 102.7 -> 103.7 mm
- net GND: vias 323 -> 321
Other:
- board text added: "Design based on MiSTeryshield PiPico USB"
- board text added: "added features and modifications by Manger"
- board text removed: "Design based on MiSTeryshield"
- board text removed: "PiPico USB : added features"
- board text removed: "and modifications by Manger"

Commit message: Add files via upload
Parts:
- D1: value TVS DIODE 5V -> SMF5.0A (TVS DIODE 5V)
Other:
- board text added: "Joystick & Mouse Port 1"
- board text removed: "Joystick Port 1"
