File: mistle_gw3a_20/usbhub.kicad_sch (KiCad schematic)
At the start: 9 parts, among them J13 USB_A_Stacked, J7 USB_A_Stacked, U12 CH334R, Y3 12MHz

Commit message: Update gw3a dev board
Parts:
- C28, C29, C30, C31, F2, J13, J7, Y3: checked once -> (none)
Changed lines of the file:
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@@
-			)
-		)
-		(property "checked" "once"
-			(at 196.85 55.88 90)
-			(hide yes)
-			(show_name no)
-			(do_not_autoplace no)
-			(effects
-				(font
-					(size 1.27 1.27)
-				)
 			)
 		)
@@
 			)
 		)
-		(property "checked" "once"
-			(at 105.41 65.405 0)
-			(hide yes)
-			(show_name no)
-			(do_not_autoplace no)
-			(effects
-				(font
-					(size 1.27 1.27)
-				)
-			)
-		)
 		(pin "1"
 		)
@@
 		)
 		(property "Comment" "Samsung 25V X5R"
-			(at 97.79 65.405 0)
-			(hide yes)
-			(show_name no)
-			(do_not_autoplace no)
-			(effects
-				(font
-					(size 1.27 1.27)
-				)
-			)
-		)
-		(property "checked" "once"
 			(at 97.79 65.405 0)
 			(hide yes)
@@
 			)
 		)
-		(property "checked" "once"
-			(at 113.03 65.405 0)
-			(hide yes)
-			(show_name no)
-			(do_not_autoplace no)
-			(effects
-				(font
-					(size 1.27 1.27)
-				)
-			)
-		)
 		(pin "1"
 		)
@@
 			)
 		)
-		(property "checked" "once"
-			(at 231.14 107.95 0)
-			(hide yes)
-			(show_name no)
-			(do_not_autoplace no)
-			(effects
-				(font
-					(size 1.27 1.27)
-				)
-			)
-		)
 		(pin "8"
 		)
@@
 			)
 		)
-		(property "checked" "once"
-			(at 90.17 65.405 0)
-			(hide yes)
-			(show_name no)
-			(do_not_autoplace no)
-			(effects
-				(font
-					(size 1.27 1.27)
-				)
-			)
-		)
 		(pin "1"
 		)
@@
 			)
 		)
-		(property "checked" "once"
-			(at 231.14 66.04 0)
-			(hide yes)
-			(show_name no)
-			(do_not_autoplace no)
-			(effects
-				(font
-					(size 1.27 1.27)
-				)
-			)
-		)
 		(pin "8"
 		)
@@
 			(at 109.22 108.585 0)
 			(hide yes)
-			(show_name no)
-			(do_not_autoplace no)
-			(effects
-				(font
-					(size 1.27 1.27)
-				)
-			)
-		)
-		(property "checked" "once"
-			(at 109.22 108.585 0)
-			(hide yes)

Commit message: Update mistle-gw3a board for rp2350
Parts:
- removed U12: CH334R, Package_SO:QSOP-16_3.9x4.9mm_P0.635mm, symbol Interface_USB:CH334R
- added U5: CH334P, Package_DFN_QFN:QFN-16-1EP_3x3mm_P0.5mm_EP1.45x1.45mm_ThermalVias, symbol ch334:CH334P
Connections:
- net +5V: now also U5.15 (V5)
- net GND: now also U5.17 (GND)
- net USB1_D+: now also U5.10 (DP1+)
- net USB1_D-: now also U5.9 (DM1-)
- net USB2_D+: now also U5.8 (DP2+)
- net USB2_D-: now also U5.7 (DM2-)
- net USB3_D+: now also U5.6 (DP3+)
- net USB3_D-: now also U5.5 (DM3-)
- net USB4_D+: now also U5.4 (DP4+)
- net USB4_D-: now also U5.3 (DM4-)
- net USB_D+: now also U5.12 (DPU+)
- net USB_D-: now also U5.11 (DMU-)
- net at C30.2, C31.2: now also U5.16 (VDD33_{LDO})
- net at Y3.1: now also U5.1 (XO)
- net at Y3.3: now also U5.2 (XI)
- no-connect marks 1 -> 2
Changed lines of the file:
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@@
+	)
+	(no_connect
+		(at 124.46 90.805)
 	)
 	(no_connect
@@
 	)
 	(symbol
+		(lib_id "ch334:CH334P")
+		(at 137.16 88.265 0)
+		(unit 1)
+		(body_style 1)
+		(exclude_from_sim no)
+		(in_bom yes)
+		(on_board yes)
+		(in_pos_files yes)
+		(dnp no)
+		(property "Reference" "U5"
+			(at 127.508 69.088 0)
+			(show_name no)
+			(do_not_autoplace no)
+			(effects
+				(font
+					(size 1.27 1.27)
+				)
+				(justify left)
+			)
+		)
+		(property "Value" "CH334P"
+			(at 143.002 107.696 0)
+			(show_name no)
+			(do_not_autoplace no)
+			(effects
+				(font
+					(size 1.27 1.27)
+				)
+			)
+		)
+		(property "Footprint" "Package_DFN_QFN:QFN-16-1EP_3x3mm_P0.5mm_EP1.45x1.45mm_ThermalVias"
+			(at 137.16 88.265 0)
+			(hide yes)
+			(show_name no)
+			(do_not_autoplace no)
+			(effects
+				(font
+					(size 1.27 1.27)
+				)
+			)
+		)
+		(property "Datasheet" ""
+			(at 137.16 88.265 0)
+			(hide yes)
+			(show_name no)
+			(do_not_autoplace no)
+			(effects
+				(font
+					(size 1.27 1.27)
+				)
+			)
+		)
+		(property "Description" ""
+			(at 137.16 88.265 0)
+			(hide yes)
+			(show_name no)
+			(do_not_autoplace no)
+			(effects
+				(font
+					(size 1.27 1.27)
+				)
+			)
+		)
+		(property "LCSC Part #" "C5373042"
+			(at 137.16 88.265 0)
+			(hide yes)
+			(show_name no)
+			(do_not_autoplace no)
+			(effects
+				(font
+					(size 1.27 1.27)
+				)
+			)
+		)
+		(property "FT Rotation Offset" "180"
+			(at 137.16 88.265 0)
+			(hide yes)
+			(show_name no)
+			(do_not_autoplace no)
+			(effects
+				(font
+					(size 1.27 1.27)
+				)
+			)
+		)
+		(pin "13"
+		)
+		(pin "12"
+		)
+		(pin "17"
+		)
+		(pin "11"
+		)
+		(pin "8"
+		)
+		(pin "7"
+		)
+		(pin "6"
+		)
+		(pin "3"
+		)
+		(pin "2"
+		)
+		(pin "1"
+		)
+		(pin "5"
+		)
+		(pin "4"
+		)
+		(pin "15"
+		)
+		(pin "16"
+		)
+		(pin "9"
+		)
+		(pin "14"
+		)
+		(pin "10"
+		)
+		(instances
+			(project "mistle_gw3a_20"
+				(path "/ba62e47e-9e07-4e97-ab08-24b670d50f97/9977593d-13fc-49aa-acc2-4d950fd30b3e"
+					(reference "U5")
+					(unit 1)
+				)
+			)
+		)
+	)
+	(symbol
 		(lib_id "Device:C_Small")
 		(at 113.03 65.405 180)
@@
 					(unit 1)
 				)
-			)
-		)
-	)
-	(symbol
-		(lib_id "Interface_USB:CH334R")
-		(at 137.16 88.265 0)
-		(unit 1)
-		(body_style 1)
-		(exclude_from_sim no)
-		(in_bom yes)
-		(on_board yes)
-		(in_pos_files yes)
-		(dnp no)
-		(property "Reference" "U12"
-			(at 139.3033 107.95 0)
-			(show_name no)
-			(do_not_autoplace no)
-			(effects
-				(font
-					(size 1.27 1.27)
-				)
-				(justify left)
-			)
-		)
-		(property "Value" "CH334R"
-			(at 139.3033 110.49 0)
-			(show_name no)
-			(do_not_autoplace no)
-			(effects
-				(font
-					(size 1.27 1.27)
-				)
-				(justify left)
-			)
-		)
-		(property "Footprint" "Package_SO:QSOP-16_3.9x4.9mm_P0.635mm"
-			(at 139.7 111.125 0)
-			(hide yes)
-			(show_name no)
-			(do_not_autoplace no)
-			(effects
-				(font
-					(size 1.27 1.27)
-				)
-				(justify left)
-			)
-		)
-		(property "Datasheet" "https://www.wch-ic.com/downloads/file/327.html"
-			(at 137.16 55.245 0)
-			(hide yes)
-			(show_name no)
-			(do_not_autoplace no)
-			(effects
-				(font
-					(size 1.27 1.27)
-				)
-			)
-		)
-		(property "Description" "USB HUB controller, QSOP-16"
-			(at 137.16 88.265 0)
-			(hide yes)
-			(show_name no)
-			(do_not_autoplace no)
-			(effects
-				(font
-					(size 1.27 1.27)
-				)
-			)
-		)
-		(property "LCSC Part #" "C4154405"
-			(at 137.16 88.265 0)
-			(hide yes)
-			(show_name no)
-			(do_not_autoplace no)
-			(effects
-				(font
-					(size 1.27 1.27)
-				)
-			)
-		)
-		(property "FT Rotation Offset" "270"
-			(at 137.16 88.265 0)
-			(hide yes)
-			(show_name no)
-			(do_not_autoplace no)
-			(effects
-				(font
-					(size 1.27 1.27)
-				)
-			)
-		)
-		(pin "10"
-		)
-		(pin "11"
-		)
-		(pin "9"
-		)
-		(pin "13"
-		)
-		(pin "16"
-		)
-		(pin "15"
-		)
-		(pin "7"
-		)
-		(pin "2"
-		)
-		(pin "4"
-		)
-		(pin "3"
-		)
-		(pin "14"
-		)
-		(pin "6"
-		)
-		(pin "5"
-		)
-		(pin "8"
-		)
-		(pin "1"
-		)
-		(pin "12"
-		)
-		(instances
-			(project "mistle_gw3a_20"
-				(path "/ba62e47e-9e07-4e97-ab08-24b670d50f97/9977593d-13fc-49aa-acc2-4d950fd30b3e"
-					(reference "U12")
-					(unit 1)
-				)
