File: mistle_gw3a_20/gw3a-lv20.kicad_sch (KiCad schematic)
At the start: 48 parts, among them J3 Jumper block, U8 SY8113BADC, Y2 50MHz

Commit message: Update gw3a dev board
Parts:
- removed R22: 10k, Resistor_SMD:R_0402_1005Metric, symbol Device:R_Small
- removed unit 9 of U7
- removed unit 10 of U7
Connections:
- net +1V0: no longer C37.2, C38.1, C39.1, C62.1, C63.2, C64.2, C65.1, C66.1, L1.2, R39.2
- net +3.3V: now also U7.100 (VCCIO7), U7.103 (VCCIO7), U7.109 (VCCIO10_VCCX), U7.117 (VCCIO6), U7.12 (VCCIO4), U7.127 (VCCIO6), U7.132 (VCCIO6), U7.18 (VCCIO4), U7.26 (VCCIO4), U7.31 (VCCIO3), U7.33 (VCCIO3), U7.40 (VCCIO10_VCCX), U7.5 (VCCIO5), U7.51 (VCCIO2), U7.55 (VCCIO2), U7.63 (VCCIO2), U7.70 (VCCIO10_VCCX), U7.77 (VCCIO1), U7.9 (VCCIO5), U7.91 (VCCIO0)
- net +0V9: now reaches U7.1 (VCC)
- net +0V9: now also C37.2, C38.1, C39.1, C62.1, C63.2, C64.2, C65.1, C66.1, L1.2, R39.2, U7.108 (VCC), U7.110 (VCC), U7.138 (VCC), U7.36 (VCC), U7.38 (VCC), U7.73 (VCC), U7.81 (VCC)
- no-connect marks 5 -> 4
Other:
- sheet Interfaces ports: added none; removed CK+, CK-, D0+, D0-, D1+, D1-, D2+, D2-, JOYA[0..5], JOYB[0..5], KEY[0..1], LED[0..5], WS2812
- note added: "DS1351 3.1.2: eFuse voltage 1.62-1.98V if efuse writing is needed. Can be left open otherwise"
- note added: "TODO: 3.1.5: What's meant by Power On Reset Voltage"
- moved on the sheet: C15, C16, C17, C4, C41, C42, C43, C44, C46, C47, C48, C49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

Commit message: Update gw3a 20 dev board
Parts:
- removed J3: Jumper block, Connector_PinHeader_2.54mm:PinHeader_2x06_P2.54mm_Vertical, symbol Connector_Generic:Conn_02x06_Odd_Even
- removed JP11: DO, Jumper:SolderJumper-2_P1.3mm_Bridged_RoundedPad1.0x1.5mm, symbol Jumper:SolderJumper_2_Bridged
- removed JP12: DI, Jumper:SolderJumper-2_P1.3mm_Bridged_RoundedPad1.0x1.5mm, symbol Jumper:SolderJumper_2_Bridged
- removed JP13: CLK, Jumper:SolderJumper-2_P1.3mm_Bridged_RoundedPad1.0x1.5mm, symbol Jumper:SolderJumper_2_Bridged
- removed JP14: ~{CS}, Jumper:SolderJumper-2_P1.3mm_Bridged_RoundedPad1.0x1.5mm, symbol Jumper:SolderJumper_2_Bridged
- removed R40: 4k7, Resistor_SMD:R_0402_1005Metric, symbol Device:R_Small
- added J3: JTAG, Connector_PinHeader_2.54mm:PinHeader_1x06_P2.54mm_Vertical, symbol Connector:Conn_01x06_Pin
- C41, C42, C43, C44, FB3, FB4: now not fitted; now left out of the parts list
- C65, C66, C67, C68: now fitted
Connections:
- net +1V0 is gone; now on net +0.9V: FB3.1, FB4.1
- net GND: now also J3.6 (Pin_6)
- net Interfaces/SD_CLK: now also R26.1
- net TCK: now also R18.1, U7.71 (TCK), J3.2 (Pin_2)
- net TDI: now also U7.72 (TDI), J3.3 (Pin_3)
- net TDO: now also R19.2, U7.69 (TDO), J3.4 (Pin_4)
- net TMS: now also U7.68 (TMS), J3.1 (Pin_1)
- net ~{CFG}: now also J3.5 (Pin_5)
- net +0V9 renamed +0.9V
- net CLK50 renamed Interfaces/CLK50
Other:
- sheet Interfaces ports: added SD_CMD; removed none
- note added: "Pinout considerations - MSPI ~{WP}/~{HOLD} wired to D02 and D03 for optional QSPI - LVDS only available in banks 2 and 6 - If SDRAM is powered at != 3.3V, then this voltage must also work for the flash - Buttons to MODE0/MODE1 as on the TN20k - SD card power switch? - Wire 4-bit SDIO to rp2040?"
- note removed: "Option to disconnect the FPGA's JTAG from the RP2040 MCU"
- note removed: "Option to disconnect the SD card from the RP2040 MCU"
- note removed: "Pinout considerations - MSPI ~{WP}/~{HOLD} wired to D02 and D03 for optional QSPI - LVDS only available in banks 2 and 6 - If SDRAM is powered at != 3.3V, then this voltage must also work for the flash - TODO: Connect buttons to MODE0/MODE1 as on the TN20k - TODO: Wire 4-bit SDIO to rp2040"
- moved on the sheet: C15, C16, C17, C64, R17, R18, R19, R26, Y2

Commit message: Update gw3a dev board
Parts:
- C15, C16, C17, C33, C34, C35, C36, C37, C38, C39, C4, C41, C42, C43, C44, C46, C47, C48, C49, C50, C62, C63, C64, FB3, FB4, L1, R17, R18, R19, R26, R38, R39, R56, U8: checked once -> (none)
- C65, C66, C67, C68: footprint Capacitor_SMD:C_0603_1608Metric -> Capacitor_SMD:C_0402_1005Metric; LCSC Part # C14663 -> C1525; checked once -> (none); now in the parts list
- J3: now left out of the parts list
- R37: LCSC Part # C11702 -> C25792; checked once -> (none)
- U7: value (none) -> GW3A-LV20-Q144
- Y2: LCSC Part # (none) -> C2901592; checked once -> (none)

Commit message: Update gw3a board
Parts:
- removed C41, C43: 10uF, Capacitor_SMD:C_0402_1005Metric, symbol Device:C_Small
- removed C42, C44: 100nF, Capacitor_SMD:C_0402_1005Metric, symbol Device:C_Small
- removed FB3, FB4: MPZ1608S101, Inductor_SMD:L_0603_1608Metric, symbol Device:FerriteBead
- added R22: 1k, Resistor_SMD:R_0402_1005Metric, symbol Device:R_Small
Connections:
- net GND: now also R22.1
- net at U7.95 (IOT29A/PUDC_B): now also R22.2
- no-connect marks 4 -> 3
Other:
- note added: "Pinout considerations - MSPI ~{WP}/~{HOLD} wired to D02 and D03 for optional QSPI - LVDS only available in banks 2 and 6 - If SDRAM is powered at != 3.3V, then this voltage must also work for the flash - Buttons to MODE0/MODE1 as on the TN20k"
- note removed: "Pinout considerations - MSPI ~{WP}/~{HOLD} wired to D02 and D03 for optional QSPI - LVDS only available in banks 2 and 6 - If SDRAM is powered at != 3.3V, then this voltage must also work for the flash - Buttons to MODE0/MODE1 as on the TN20k - SD card power switch? - Wire 4-bit SDIO to rp2040?"
- moved on the sheet: C15, R17, Y2

Commit message: Add expansion connector
Connections:
- net MON_TX: no longer names the net of U7.86 (IOT52B)
- no-connect marks 3 -> 4
Other:
- sheet Interfaces ports: added none; removed MON_RX, MON_TX
- note added: "GW5A-LV25-LQ144 compatibility - supply - vss/vccio1/2/5/6/7/10_vccx/vefuse/vcc -> ok - gw5 vccio0_4 maps to gw3 vccio0 and vccio4 -> prob ok"
Changed lines of the file:
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@@
 		)
 	)
+	(text "GW5A-LV25-LQ144 compatibility\n- supply\n  - vss/vccio1/2/5/6/7/10_vccx/vefuse/vcc -> ok\n  - gw5 vccio0_4 maps to gw3 vccio0 and vccio4 -> prob ok\n"
+		(exclude_from_sim no)
+		(at 106.68 127 0)
+		(effects
+			(font
+				(size 1.27 1.27)
+			)
+			(justify left top)
+		)
+	)
 	(text "Pinout considerations\n- MSPI ~{WP}/~{HOLD} wired to D02 and D03 for optional QSPI\n- LVDS only available in banks 2 and 6\n- If SDRAM is powered at != 3.3V, then this voltage must also work for the flash\n- Buttons to MODE0/MODE1 as on the TN20k"
 		(exclude_from_sim no)
@@
 	)
 	(junction
-		(at 115.57 98.425)
-		(diameter 0)
-		(color 0 0 0 0)
-	)
-	(junction
 		(at 115.57 75.565)
 		(diameter 0)
@@
 	)
 	(junction
+		(at 115.57 95.885)
+		(diameter 0)
+		(color 0 0 0 0)
+	)
+	(junction
 		(at 48.895 65.405)
 		(diameter 0)
@@
 	)
 	(no_connect
+		(at 53.975 114.3)
+	)
+	(no_connect
 		(at 149.86 55.245)
 	)
@@
 	(wire
 		(pts
-			(xy 53.975 114.3) (xy 48.895 114.3)
-		)
-		(stroke
-			(width 0)
-			(type default)
-		)
-	)
-	(wire
-		(pts
 			(xy 153.67 61.595) (xy 153.67 59.055)
 		)
@@
 	(wire
 		(pts
-			(xy 115.57 100.965) (xy 115.57 98.425)
-		)
-		(stroke
-			(width 0)
-			(type default)
-		)
-	)
-	(wire
-		(pts
 			(xy 23.495 174.625) (xy 29.845 174.625)
 		)
@@
 	(wire
 		(pts
-			(xy 109.22 98.425) (xy 115.57 98.425)
+			(xy 109.22 100.965) (xy 115.57 100.965)
 		)
 		(stroke
@@
 	(wire
 		(pts
-			(xy 153.67 86.995) (xy 153.67 89.535)
+			(xy 115.57 95.885) (xy 115.57 98.425)
 		)
 		(stroke
@@
 	(wire
 		(pts
-			(xy 115.57 100.965) (xy 118.11 100.965)
+			(xy 153.67 86.995) (xy 153.67 89.535)
 		)
 		(stroke
@@
 	(wire
 		(pts
-			(xy 48.895 65.405) (xy 60.325 65.405)
+			(xy 115.57 100.965) (xy 118.11 100.965)
 		)
 		(stroke
@@
 	(wire
 		(pts
-			(xy 194.31 57.785) (xy 194.31 56.515)
+			(xy 48.895 65.405) (xy 60.325 65.405)
 		)
 		(stroke
@@
 	(wire
 		(pts
-			(xy 75.565 174.625) (xy 75.565 177.165)
+			(xy 194.31 57.785) (xy 194.31 56.515)
 		)
 		(stroke
@@
 	(wire
 		(pts
-			(xy 233.045 43.815) (xy 234.95 43.815)
+			(xy 75.565 174.625) (xy 75.565 177.165)
 		)
 		(stroke
@@
 	(wire
 		(pts
-			(xy 53.975 96.52) (xy 40.005 96.52)
+			(xy 233.045 43.815) (xy 234.95 43.815)
 		)
 		(stroke
@@
 	(wire
 		(pts
-			(xy 229.87 82.55) (xy 234.95 82.55)
+			(xy 53.975 96.52) (xy 40.005 96.52)
 		)
 		(stroke
@@
 	(wire
 		(pts
-			(xy 229.87 80.01) (xy 234.95 80.01)
-		)
-		(stroke
-			(width 0)
-			(type default)
-		)
-	)
-	(wire
-		(pts
 			(xy 229.87 74.295) (xy 234.95 74.295)
 		)
@@
 		)
 	)
-	(global_label "MON_TX"
-		(shape input)
-		(at 229.87 82.55 180)
-		(fields_autoplaced yes)
-		(effects
-			(font
-				(size 1.27 1.27)
-			)
-			(justify right)
-		)
-		(property "Intersheetrefs" "${INTERSHEET_REFS}"
-			(at 220.2819 82.55 0)
-			(hide yes)
-			(show_name no)
-			(do_not_autoplace no)
-			(effects
-				(font
-					(size 1.27 1.27)
-				)
-				(justify right)
-			)
-		)
-	)
-	(global_label "MON_TX"
-		(shape output)
-		(at 48.895 114.3 180)
-		(fields_autoplaced yes)
-		(effects
-			(font
-				(size 1.27 1.27)
-			)
-			(justify right)
-		)
-		(property "Intersheetrefs" "${INTERSHEET_REFS}"
-			(at 39.3069 114.3 0)
-			(hide yes)
-			(show_name no)
-			(do_not_autoplace no)
-			(effects
-				(font
-					(size 1.27 1.27)
-				)
-				(justify right)
-			)
-		)
-	)
 	(global_label "~{CFG}"
 		(shape input)
@@
 		)
 	)
-	(global_label "MON_RX"
-		(shape output)
-		(at 229.87 80.01 180)
-		(fields_autoplaced yes)
-		(effects
-			(font
-				(size 1.27 1.27)
-			)
-			(justify right)
-		)
-		(property "Intersheetrefs" "${INTERSHEET_REFS}"
-			(at 219.9795 80.01 0)
-			(hide yes)
-			(show_name no)
-			(do_not_autoplace no)
-			(effects
-				(font
-					(size 1.27 1.27)
-				)
-				(justify right)
-			)
-		)
-	)
 	(global_label "MIDI_OUT"
 		(shape output)
@@
 		(lib_name "+3V3_1")
 		(lib_id "power:+3V3")
-		(at 109.22 98.425 90)
+		(at 109.22 100.965 90)
 		(unit 1)
 		(body_style 1)
@@
 		(dnp no)
 		(property "Reference" "#PWR069"
-			(at 113.03 98.425 0)
+			(at 113.03 100.965 0)
 			(hide yes)
 			(show_name no)
@@
 		)
 		(property "Value" "+3.3V"
-			(at 104.648 98.171 90)
+			(at 104.648 100.711 90)
 			(show_name no)
 			(do_not_autoplace no)
@@
 		)
 		(property "Footprint" ""
-			(at 109.22 98.425 0)
+			(at 109.22 100.965 0)
 			(hide yes)
 			(show_name no)
@@
 		)
 		(property "Datasheet" ""
-			(at 109.22 98.425 0)
+			(at 109.22 100.965 0)
 			(hide yes)
 			(show_name no)
@@
 		)
 		(property "Description" "Power symbol creates a global label with name \"+3V3\""
-			(at 109.22 98.425 0)
+			(at 109.22 100.965 0)
 			(hide yes)
 			(show_name no)
@@
 	(sheet
 		(at 234.95 34.925)
-		(size 26.67 50.8)
+		(size 26.67 41.91)
 		(exclude_from_sim no)
 		(in_bom yes)
@@
 		)
 		(property "Sheetfile" "interfaces.kicad_sch"
-			(at 234.95 86.3096 0)
+			(at 234.95 77.4196 0)
 			(show_name no)
 			(do_not_autoplace no)
@@
 			(effects
 				(font
-					(size 1.27 1.27)
-				)
-				(justify left)
-			)
-		)
-		(pin "MON_RX" output
-			(at 234.95 80.01 180)
-			(effects
-				(font
-					(size 1.27 1.27)
-				)
-				(justify left)
-			)
-		)
-		(pin "MON_TX" input
-			(at 234.95 82.55 180)
-			(effects
-				(font
