File: icepi_carrier/icepi_carrier.kicad_pcb (KiCad board)
At the start: 2 copper layers, 42.8 x 81.8 mm, 83 parts, among them J1 SWD, J11 DB9M, J12 DB9M, J13 USB_A_Stacked, J2 USB_C_Receptacle_USB2.0, J3 Conn_02x20_Odd_Even, J7 USB_A_Stacked, SW1 Boot, U10 74LCX07, U11 RP2350_60QFN, U2 W25Q64JVS, U3 USBLC6-2SC6, U5 CH334P, U9 74LCX07, Y1 12MHz, Y3 12MHz

Commit message: Update icepi carrier for first test production
Parts:
- D13, D7: value green -> yellow
- D14: value green -> red
- moved TP3 8.07 mm to (171.4, 82.9)
- moved TP2 4.97 mm to (171.4, 80.8)
- moved R45 4.39 mm to (184.1, 64.3)
- moved D12 4.38 mm to (186.5, 64.3)
- moved R47 4.36 mm to (184.1, 68.7)
- moved D14 4.20 mm to (186.5, 68.5)
- moved TP4 2.15 mm to (171.4, 78.7)
- moved TP1 2.14 mm to (171.4, 76.6)
- moved D13 0.08 mm to (186.5, 66.5)
Routing:
- net +5V: track 161.7 -> 147.9 mm, vias 4 -> 5
- net /Icepi-zero/DOWN-1: track 66.8 -> 60.0 mm, vias 3 -> 4
- net TDI: track 9.40 -> 14.4 mm
- net Net-(J3-Pin_10): track 42.4 -> 47.2 mm
- net TCK: track 2.85 -> 5.02 mm
- net SCK: track 22.2 -> 24.0 mm
- net GND: track 25.5 -> 23.7 mm, vias 20 -> 24
- net MISO: track 38.9 -> 40.4 mm
- net LED 2: track 31.1 -> 32.5 mm
- net LED 1: track 34.6 -> 35.9 mm
- net Net-(J13-VBUS1): track 26.7 -> 27.9 mm
- net SWD: track 21.0 -> 19.9 mm
- net TDO: track 9.39 -> 10.5 mm
- net LED 3: track 27.7 -> 28.7 mm
- net /Icepi-zero/BTN2-1: track 46.7 -> 47.6 mm
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
Commit message: Replace ws2812b with slightly bigger one
Parts:
- D5: value WS2812B-2020 -> WS2812B; footprint LED_SMD:LED_WS2812B-2020_PLCC4_2.0x2.0mm -> LED_SMD:LED_WS2812B-Mini_PLCC4_3.5x3.5mm
- moved R20 19.4 mm to (152.1, 106.4), turned to 0 degrees
- moved R21 4.95 mm to (165.0, 120.6)
- moved D5 0.82 mm to (168.4, 120.3)
- moved Y3 0.31 mm to (167.7, 115.5)
Connections:
- D5 pad 1: unconnected-(D5-DOUT-Pad1) -> +5V
- D5 pad 2: GND -> unconnected-(D5-DOUT-Pad2)
- D5 pad 3: Net-(D5-DIN) -> GND
- D5 pad 4: +5V -> Net-(D5-DIN)
Routing:
- net Net-(D5-DIN): track 7.19 -> 27.7 mm
- net Net-(J3-Pin_32): track 45.9 -> 26.4 mm
- net +5V: track 147.9 -> 155.9 mm
- net ~{CS}: track 30.1 -> 28.3 mm
Other:
- board text added: "IcePi Carrier V1.0a"
- board text removed: "IcePi Carrier V1.0"
