File: icepi_carrier/icepi_carrier.kicad_sch (KiCad schematic)
At the start: 52 parts, among them J1 SWD, J2 USB_C_Receptacle_USB2.0, SW1 Boot, U11 RP2350_60QFN, U2 W25Q64JVS, U3 USBLC6-2SC6, Y1 12MHz

Commit message: Update icepi carrier for first test production
Parts:
- D7: value green -> yellow; LCSC Part # C2297 -> C2296
Changed lines of the file:
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@@
 			)
 		)
-		(property "Value" "green"
+		(property "Value" "yellow"
 			(at 138.43 157.861 0)
 			(show_name no)
@@
 			)
 		)
-		(property "LCSC Part #" "C2297"
+		(property "LCSC Part #" "C2296"
 			(at 133.985 163.195 0)
 			(hide yes)
