File: icepi_carrier/icepi_zero.kicad_sch (KiCad schematic)
At the start: 22 parts, among them J11 DB9M, J12 DB9M, J3 Conn_02x20_Odd_Even, U10 74LCX07, U9 74LCX07

Commit message: Update icepi carrier for first test production
Parts:
- D13: value green -> yellow; LCSC Part # C2297 -> C2296
- D14: value green -> red; LCSC Part # C2297 -> C2295
Changed lines of the file:
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@@
 			)
 		)
-		(property "Value" "green"
+		(property "Value" "yellow"
 			(at 103.886 130.81 0)
 			(show_name no)
@@
 			)
 		)
-		(property "LCSC Part #" "C2297"
+		(property "LCSC Part #" "C2296"
 			(at 104.14 133.35 0)
 			(hide yes)
@@
 			)
 		)
-		(property "Value" "green"
+		(property "Value" "red"
 			(at 103.886 137.922 0)
 			(show_name no)
@@
 			)
 		)
-		(property "LCSC Part #" "C2297"
+		(property "LCSC Part #" "C2295"
 			(at 104.14 140.335 0)
 			(hide yes)

Commit message: Replace ws2812b with slightly bigger one
Parts:
- D5: value WS2812B-2020 -> WS2812B; footprint LED_SMD:LED_WS2812B-2020_PLCC4_2.0x2.0mm -> LED_SMD:LED_WS2812B-Mini_PLCC4_3.5x3.5mm; symbol LED:WS2812B-2020 -> LED:WS2812B; LCSC Part # C965555 -> C527089
Connections:
- net +5V: now also D5.1 (VDD); no longer D5.4 (VDD)
- net GND: now also D5.3 (VSS); no longer D5.2 (VSS)
- net at R20.2, R21.2: now also D5.4 (DIN); no longer D5.3 (DIN)
Changed lines of the file:
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@@
 		(title "MiSTle IcePi Carrier")
 		(date "2026-04-29")
-		(rev "1.0")
+		(rev "1.0a")
 		(company "Till Harbaum")
 		(comment 1 "IcePi-Zero")
@@
 	)
 	(symbol
-		(lib_id "LED:WS2812B-2020")
+		(lib_id "LED:WS2812B")
 		(at 154.94 142.875 0)
 		(unit 1)
@@
 			)
 		)
-		(property "Value" "WS2812B-2020"
+		(property "Value" "WS2812B"
 			(at 144.78 135.255 0)
 			(show_name no)
@@
 			)
 		)
-		(property "Footprint" "LED_SMD:LED_WS2812B-2020_PLCC4_2.0x2.0mm"
+		(property "Footprint" "LED_SMD:LED_WS2812B-Mini_PLCC4_3.5x3.5mm"
 			(at 156.21 150.495 0)
 			(hide yes)
@@
 			)
 		)
-		(property "Datasheet" "https://cdn-shop.adafruit.com/product-files/4684/4684_WS2812B-2020_V1.3_EN.pdf"
+		(property "Datasheet" "https://cdn-shop.adafruit.com/datasheets/WS2812B.pdf"
 			(at 157.48 152.4 0)
 			(hide yes)
@@
 			)
 		)
-		(property "Description" "RGB LED with integrated controller, 2.0 x 2.0 mm, 12 mA"
+		(property "Description" "RGB LED with integrated controller"
 			(at 154.94 142.875 0)
 			(hide yes)
@@
 			)
 		)
-		(property "LCSC Part #" "C965555"
+		(property "LCSC Part #" "C527089"
 			(at 154.94 142.875 0)
 			(hide yes)
